File: HandyRadio/HW/V1_09302022/1- Design Files/_HW_HandyRadio_/[06] - DCDC PWS.kicad_sch (KiCad schematic)
At the start: 0 parts

Commit message: 2/6 HandyRadio HW has been done
Parts:
- added C? (x4): 100nF, symbol HandyRadio:100nF
- added EC? (x2): 4u7F/6.3V, symbol HandyRadio:4u7F{brace}slash}6.3V
- added EC? (x2): 2u2F/10V, symbol HandyRadio:2u2F/10V
- added R?: 10KR, symbol HandyRadio:10KR
- added U?: MIC5365-3.3, symbol HandyRadio:MIC5365-3.3
Connections:
- new net: R?.2, U?.3 (EN)
- new net +3.3V: C?.2, EC?.1, U?.5 (VOUT)
- new net +5V: C?.2, EC?.1, R?.1, U?.1 (VIN)
- new net GND: C?.1, C?.1, EC?.2, EC?.2, U?.2 (GND)
Other:
- note added: "Duty Cycle = (1-Vi/Vo) = (1-(3.7/7.5)) ~= 50% fGate = fOSC/2 => fOSC = 1 / (4 * Rfreq * 4.75pF) ==> Rfreq = 260 KR fOSC = 202,429 Hz fGate = 101,214 Hz Ipeak = (3.7 * 0.5) / (10uH * fGate) = 1.83 A"

Commit message: power supply section has been done
Parts:
- added C?: 680pF, symbol HandyRadio:680pF
- added C? (x6): 4u7F, symbol HandyRadio:4u7F
- added C?: 220nF, symbol HandyRadio:220nF
- added D?: DSS13U, symbol HandyRadio:DSS13U
- added EC? (x2): 2u2F/10V, symbol HandyRadio:2u2F/10V
- added EC?: 4u7F/6.3V, symbol HandyRadio:4u7F{brace}slash}6.3V
- added J?: XH_CONN_2POS_R/A, symbol HandyRadio:XH_CONN_2POS_R/A
- added J?: USB_uAB_RECEP, symbol HandyRadio:USB_uAB_RECEP
- added L?: 10uH, symbol HandyRadio:10uH
- added Q?: IRF7401TRPBF, symbol HandyRadio:IRF7401TRPBF
- added R? (x2): 100KR, symbol HandyRadio:100KR
- added R?: POT_5KR, symbol HandyRadio:POT_5KR
- added R? (x2): 2KR, symbol HandyRadio:2KR
- added R?: 10KR, symbol HandyRadio:10KR
- added R?: 30KR, symbol HandyRadio:30KR
- added R?: 16KR5, symbol HandyRadio:16KR5
- added R?: 82KR, symbol HandyRadio:82KR
- added U?: MCP73831, symbol HandyRadio:MCP73831
- added U?: AP7361EA, symbol HandyRadio:AP7361EA
- added U?: R1211N002B, symbol HandyRadio:R1211N002B
Connections:
- net +5V: now also C?.2, EC?.1, U?.1 (OUT)
- net GND: now also C?.1, C?.1, EC?.2, EC?.2, C?.1, C?.1, C?.1, C?.1, C?.1, C?.1, C?.2, EC?.2, EC?.2, EC?.2, J?.2, J?.5 (GND), Q?.1 (S), Q?.2 (S), Q?.3 (S), R?.1, R?.3, U?.2 (VSS), U?.4 (GND), U?.5 (VFB)
- net +6V: now reaches C?.2
- net +6V: now also EC?.1, C?.1, C?.2, C?.2, D?.2, EC?.1, EC?.1, R?.1, R?.2, U?.8 (VIN)
- new net: R?.2, U?.2 (EN)
- new net: R?.1, R?.1, R?.2
- new net: Q?.4 (G), U?.6 (EXT)
- new net: D?.1, L?.2, Q?.5 (D), Q?.6 (D), Q?.7 (D), Q?.8 (D)
- new net: C?.2, J?.1 (VBUS), R?.1, U?.4 (VDD)
- new net: R?.2, U?.5 (PROG)
- new net: R?.1, R?.2
- new net: C?.1, R?.1, R?.2, R?.2, R?.2
- new net: R?.1, U?.5 (VFB)
- new net: C?.2, C?.2, C?.2, EC?.1, J?.1, L?.1, R?.1, U?.3 (VBAT), U?.4 (VIN)
- new net: R?.2, U?.2 (CE)
- new net: C?.2, U?.1 (DELAY)
- new net BATT_STAT: U?.1 (STAT)
- no-connect marks 0 -> 3
Other:
- note added: "DNF"
- note removed: "Duty Cycle = (1-Vi/Vo) = (1-(3.7/7.5)) ~= 50% fGate = fOSC/2 => fOSC = 1 / (4 * Rfreq * 4.75pF) ==> Rfreq = 260 KR fOSC = 202,429 Hz fGate = 101,214 Hz Ipeak = (3.7 * 0.5) / (10uH * fGate) = 1.83 A"
- moved on the sheet: C?, EC?, R?, U?

Commit message: Schematic is almost Done
Parts:
- removed EC?: 4u7F/6.3V, symbol HandyRadio:4u7F{brace}slash}6.3V
- removed EC?: 2u2F/10V, symbol HandyRadio:2u2F/10V
- added C? (x9): 1uF, symbol HandyRadio:1uF
- added C?: 4u7F, symbol HandyRadio:4u7F
- added EC?: 4u7F/6.3V, symbol HandyRadio:4u7F{brace}slash}6.3V
- added TP? (x9): TPC, symbol HandyRadio:TPC
Connections:
- net +3.3V: now also TP?.1
- net +5V: now also C?.1, C?.1, C?.1, C?.1, C?.1, TP?.1
- net +6V: now also C?.1, C?.1, C?.1, C?.1, TP?.1
- net GND: now also C?.1, C?.2, C?.2, C?.2, C?.2, C?.2, C?.2, C?.2, C?.2, C?.2, EC?.2, TP?.1, TP?.1, TP?.1, TP?.1
- net at C?.2, J?.1 (VBUS), R?.1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: now also C?.2
- net at C?.1, R?.1, R?.2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: now also TP?.1
- net +BATT: now reaches C?.2, C?.2, C?.2, EC?.1, J?.1, L?.1, R?.1, U?.3 (VBAT), U?.4 (VIN)
- net +BATT: now also EC?.1, TP?.1
- net DELAY: now reaches C?.2, U?.1 (DELAY)
Other:
- note added: "BATTERY"
- note added: "CAUTIONARY:"
- note added: "CHARGER"
- note added: "DC-DC BOOST"
- note added: "DO NOT FIT"
- note added: "For optimum voltage regulation, place the battery pack as close as possible to the device’s VBAT and VSS pins. This is recommended to minimize voltage drops along the high current-carrying PCB traces."
- note added: "INFO:"
- note added: "If the PCB layout is used as a heat sink, adding many vias in the heat sink pad can help conduct more heat to the PCB backplane, thus reducing the maximum junction temperature."
- note added: "LAYOUT:"
- note added: "LDO +3V3DC"
- note added: "LDO +5VDC"
- note added: "ONLY IF THE OUTPUT VOLTAGE WAS WRONG ADJUST IT WITH THESE RESISTORS"
- note added: "Output Voltage = VFB x (R1 + R2) / R2 R1 + R2 = 100 KR is recommended range of resistances VFB = @VIN = 3.3V / 0.985 ~ 1.015V"
- note added: "This input capacitor must be located as close as possible to the device to ensure input stability and reduced noise. For PCB layout, a wide copper trace is required for both the IN and GND pins."
- note added: "connect C2 between Delay pin and GND pin of the IC with the minimum wiring distance"
- note added: "• Connect a 1 µF or more value of capacitor between VOUT and GND, C3 as shown in typical applications of the previous page. (Recommended value is from 10 µF to 22 µF.) If the operation of the composed DC/DC converter may be unstable, use a tantalum type capacitor instead of ceramic type."
- company: (none) -> Siavash Taher Parvar
- title: (none) -> Handy Radio
- moved on the sheet: C?, D?, EC?, J?, L?, Q?, R?, U?

Commit message: 95 SCHEMATIC HAS BEEN DONE
Parts:
- gave numbers to parts that had none: 56

Commit message: Schematic has been double checked
Other:
- moved on the sheet: D3
Changed lines of the file:
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@@
     (stroke (width 0) (type default) (color 0 0 0 0))
   )
-  (polyline (pts (xy 355.6 128.27) (xy 394.97 128.27))
+  (polyline (pts (xy 355.6 128.27) (xy 396.24 128.27))
     (stroke (width 0) (type default) (color 0 0 0 0))
   )
@@
     (stroke (width 0) (type default) (color 0 0 0 0))
   )
-  (wire (pts (xy 264.16 87.63) (xy 267.97 87.63))
+  (wire (pts (xy 266.7 87.63) (xy 267.97 87.63))
     (stroke (width 0) (type default) (color 0 0 0 0))
   )
@@
     (stroke (width 0) (type default) (color 0 0 0 0))
   )
-  (polyline (pts (xy 394.97 128.27) (xy 394.97 148.59))
+  (polyline (pts (xy 396.24 128.27) (xy 396.24 148.59))
     (stroke (width 0) (type default) (color 0 0 0 0))
   )
@@
     (stroke (width 0) (type default) (color 0 0 0 0))
   )
-  (polyline (pts (xy 394.97 148.59) (xy 355.6 148.59))
+  (polyline (pts (xy 396.24 148.59) (xy 355.6 148.59))
     (stroke (width 0) (type default) (color 0 0 0 0))
   )
-  (wire (pts (xy 295.91 80.01) (xy 299.72 80.01))
+  (wire (pts (xy 295.91 80.01) (xy 304.8 80.01))
     (stroke (width 0) (type default) (color 0 0 0 0))
   )
@@
     (stroke (width 0) (type default) (color 0 0 0 0))
   )
-  (wire (pts (xy 325.12 80.01) (xy 312.42 80.01))
+  (wire (pts (xy 325.12 80.01) (xy 317.5 80.01))
     (stroke (width 0) (type default) (color 0 0 0 0))
   )
@@
   )
   (text "Output Voltage = \nVFB x (R1 + R2) / R2\nR1 + R2 = 100 KR is \nrecommended range of \nresistances\n\nVFB = @VIN = 3.3V / 0.985 ~ 1.015V"
-    (at 356.87 147.32 0)
+    (at 358.14 147.32 0)
     (effects (font (size 1.27 1.27)) (justify left bottom))
   )
@@
     (pin "8")
   )
-  (symbol (lib_id "HandyRadio:DSS13U") (at 299.72 80.01 0) (unit 1)
+  (symbol (lib_id "HandyRadio:DSS13U") (at 304.8 80.01 0) (unit 1)
     (in_bom yes) (on_board yes)
-    (property "Reference" "D3" (id 0) (at 313.69 78.74 0))
-    (property "Value" "DSS13U" (id 1) (at 297.18 78.74 0))
-    (property "Footprint" "" (id 2) (at 303.53 74.93 0)
+    (property "Reference" "D3" (id 0) (at 318.77 78.74 0))
+    (property "Value" "DSS13U" (id 1) (at 302.26 78.74 0))
+    (property "Footprint" "" (id 2) (at 308.61 74.93 0)
       (effects (font (size 1.27 1.27)) hide)
     )
-    (property "Datasheet" "https://www.smc-diodes.com/propdf/DSS12U%20THRU%20DSS125U%20N1873%20REV.A.pdf" (id 3) (at 306.07 72.39 0)
+    (property "Datasheet" "https://www.smc-diodes.com/propdf/DSS12U%20THRU%20DSS125U%20N1873%20REV.A.pdf" (id 3) (at 311.15 72.39 0)
       (effects (font (size 1.27 1.27)) hide)
     )
-    (property "Description" "SCHOTTKY 30V SOD-123FL" (id 4) (at 308.61 69.85 0)
+    (property "Description" "SCHOTTKY 30V SOD-123FL" (id 4) (at 313.69 69.85 0)
       (effects (font (size 1.27 1.27)) hide)
     )
@@
     (pin "2")
   )
-  (symbol (lib_id "power:GND") (at 264.16 87.63 270) (unit 1)
+  (symbol (lib_id "power:GND") (at 266.7 87.63 270) (unit 1)
     (in_bom yes) (on_board yes) (fields_autoplaced)
-    (property "Reference" "#PWR060" (id 0) (at 257.81 87.63 0)
+    (property "Reference" "#PWR060" (id 0) (at 260.35 87.63 0)
       (effects (font (size 1.27 1.27)) hide)
     )
-    (property "Value" "GND" (id 1) (at 260.35 87.6299 90)
+    (property "Value" "GND" (id 1) (at 262.89 87.6299 90)
       (effects (font (size 1.27 1.27)) (justify right))
     )
-    (property "Footprint" "" (id 2) (at 264.16 87.63 0)
+    (property "Footprint" "" (id 2) (at 266.7 87.63 0)
       (effects (font (size 1.27 1.27)) hide)
     )
-    (property "Datasheet" "" (id 3) (at 264.16 87.63 0)
+    (property "Datasheet" "" (id 3) (at 266.7 87.63 0)
       (effects (font (size 1.27 1.27)) hide)
     )

Commit message: 99% SCHEMATIC HAS BEEN DONE
Parts:
- renumbered C39 to C41, C40 to C42, C41 to C43, C42 to C44, C43 to C45, C44 to C46, C45 to C47, C46 to C48, C47 to C49, C48 to C50, C49 to C51, C50 to C52, C51 to C53, C52 to C54, C53 to C55, C54 to C56, C55 to C57, C56 to C58, C57 to C59, C58 to C60, C59 to C61, C60 to C62, R27 to R31, R28 to R32, R29 to R33, R30 to R34, R31 to R35, R32 to R36, R33 to R37, R34 to R38, R35 to R39, R36 to R40, TP12 to TP13, TP13 to TP14, TP14 to TP15, TP15 to TP16, TP16 to TP17, TP17 to TP18, TP18 to TP19, TP19 to TP20, TP20 to TP21

Commit message: footprints have been added
Parts:
- U8: footprint (none) -> Relay_THT:Relay_DPDT_AXICOM_IMSeries_Pitch5.08mm
Changed lines of the file:
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@@
     (property "Reference" "U8" (id 0) (at 259.08 92.71 0))
     (property "Value" "R1211N002B" (id 1) (at 259.08 95.25 0))
-    (property "Footprint" "" (id 2) (at 270.51 80.01 0)
+    (property "Footprint" "Relay_THT:Relay_DPDT_AXICOM_IMSeries_Pitch5.08mm" (id 2) (at 270.51 80.01 0)
       (effects (font (size 1.27 1.27)) hide)
     )
