File: HandyRadio/HW/V1_09302022/1- Design Files/_HW_HandyRadio_/[06] - DCDC PWS.kicad_sch (KiCad schematic)
At the start: 56 parts, among them J5 USB_uAB_RECEP, J6 XH_CONN_2POS_R/A, Q2 IRF7401TRPBF, U6 MCP73831, U7 AP7361EA, U8 R1211N002B, U9 MIC5365-3.3

Commit message: almost ready for routing and finishing PCB :D
Parts:
- removed EC10, EC11, EC14: 4u7F/6.3V, symbol HandyRadio:4u7F{brace}slash}6.3V
- removed EC12, EC13, EC15: 2u2F/10V, symbol HandyRadio:2u2F/10V
- added EC? (x3): 4u7F/6.3V, Capacitor_Tantalum_SMD:CP_EIA-2012-12_Kemet-R_Pad1.30x1.05mm_HandSolder, symbol HandyRadio:4u7F/6.3V
- added EC? (x3): 2u2F/10V, Capacitor_Tantalum_SMD:CP_EIA-2012-12_Kemet-R_Pad1.30x1.05mm_HandSolder, symbol HandyRadio:2u2F{brace}slash}10V
- C?: renamed from C60; footprint (none) -> Capacitor_SMD:C_0805_2012Metric_Pad1.18x1.45mm_HandSolder
- C?: renamed from C45; footprint (none) -> Capacitor_SMD:C_0805_2012Metric_Pad1.18x1.45mm_HandSolder
- C?: renamed from C50; footprint (none) -> Capacitor_SMD:C_0805_2012Metric_Pad1.18x1.45mm_HandSolder
- C?: renamed from C52; footprint (none) -> Capacitor_SMD:C_0805_2012Metric_Pad1.18x1.45mm_HandSolder
- C?: renamed from C41; footprint (none) -> Capacitor_SMD:C_0805_2012Metric_Pad1.18x1.45mm_HandSolder
- C?: renamed from C54; footprint (none) -> Capacitor_SMD:C_0805_2012Metric_Pad1.18x1.45mm_HandSolder
- C?: renamed from C47; footprint (none) -> Capacitor_SMD:C_0805_2012Metric_Pad1.18x1.45mm_HandSolder
- C?: renamed from C59; footprint (none) -> Capacitor_SMD:C_0805_2012Metric_Pad1.18x1.45mm_HandSolder
- C?: renamed from C53; footprint (none) -> Capacitor_SMD:C_0805_2012Metric_Pad1.18x1.45mm_HandSolder
- C?: renamed from C56; footprint (none) -> Capacitor_SMD:C_0805_2012Metric_Pad1.18x1.45mm_HandSolder
- C?: renamed from C49; footprint (none) -> Capacitor_SMD:C_0805_2012Metric_Pad1.18x1.45mm_HandSolder
- C?: renamed from C42; footprint (none) -> Capacitor_SMD:C_0805_2012Metric_Pad1.18x1.45mm_HandSolder
- C?: renamed from C62; footprint (none) -> Capacitor_SMD:C_0805_2012Metric_Pad1.18x1.45mm_HandSolder
- C?: renamed from C57; footprint (none) -> Capacitor_SMD:C_0805_2012Metric_Pad1.18x1.45mm_HandSolder
- C?: renamed from C44; footprint (none) -> Capacitor_SMD:C_0805_2012Metric_Pad1.18x1.45mm_HandSolder
- C?: renamed from C43; footprint (none) -> Capacitor_SMD:C_0805_2012Metric_Pad1.18x1.45mm_HandSolder
- C?: renamed from C51; footprint (none) -> Capacitor_SMD:C_0805_2012Metric_Pad1.18x1.45mm_HandSolder
- C?: renamed from C58; footprint (none) -> Capacitor_SMD:C_0805_2012Metric_Pad1.18x1.45mm_HandSolder
- C?: renamed from C48; footprint (none) -> Capacitor_SMD:C_0805_2012Metric_Pad1.18x1.45mm_HandSolder
- C?: renamed from C61; footprint (none) -> Capacitor_SMD:C_0805_2012Metric_Pad1.18x1.45mm_HandSolder
- C?: renamed from C46; footprint (none) -> Capacitor_SMD:C_0805_2012Metric_Pad1.18x1.45mm_HandSolder
- C?: renamed from C55; footprint (none) -> Capacitor_SMD:C_0805_2012Metric_Pad1.18x1.45mm_HandSolder
- D?: renamed from D3; footprint (none) -> Diode_SMD:D_SOD-123F
- J?: renamed from J6; footprint (none) -> Connector_JST:JST_PH_S2B-PH-K_1x02_P2.00mm_Horizontal
- J?: renamed from J5; footprint (none) -> Connector_USB:USB_Micro-AB_Molex_47590-0001
- L?: renamed from L5; footprint (none) -> Inductor_SMD:L_Bourns-SRN4018
- Q?: renamed from Q2; footprint (none) -> Package_SO:SOIC-8_3.9x4.9mm_P1.27mm
- R?: renamed from R32; footprint (none) -> Resistor_SMD:R_0805_2012Metric_Pad1.20x1.40mm_HandSolder
- R?: renamed from R38; footprint (none) -> Potentiometer_SMD:Potentiometer_Bourns_TC33X_Vertical
- R?: renamed from R31; footprint (none) -> Resistor_SMD:R_0805_2012Metric_Pad1.20x1.40mm_HandSolder
- R?: renamed from R36; footprint (none) -> Resistor_SMD:R_0805_2012Metric_Pad1.20x1.40mm_HandSolder
- R?: renamed from R34; footprint (none) -> Resistor_SMD:R_0805_2012Metric_Pad1.20x1.40mm_HandSolder
- R?: renamed from R40; footprint (none) -> Resistor_SMD:R_0805_2012Metric_Pad1.20x1.40mm_HandSolder
- R?: renamed from R33; footprint (none) -> Resistor_SMD:R_0805_2012Metric_Pad1.20x1.40mm_HandSolder
- R?: renamed from R39; footprint (none) -> Resistor_SMD:R_0805_2012Metric_Pad1.20x1.40mm_HandSolder
- R?: renamed from R35; footprint (none) -> Resistor_SMD:R_0805_2012Metric_Pad1.20x1.40mm_HandSolder
- R?: renamed from R37; footprint (none) -> Resistor_SMD:R_0805_2012Metric_Pad1.20x1.40mm_HandSolder
- TP?: renamed from TP19; footprint (none) -> TestPoint:TestPoint_Pad_D1.5mm
- TP?: renamed from TP13; footprint (none) -> TestPoint:TestPoint_Pad_D1.5mm
- TP?: renamed from TP18; footprint (none) -> TestPoint:TestPoint_Pad_D1.5mm
- TP?: renamed from TP20; footprint (none) -> TestPoint:TestPoint_Pad_D1.5mm
- TP?: renamed from TP16; footprint (none) -> TestPoint:TestPoint_Pad_D1.5mm
- TP?: renamed from TP21; footprint (none) -> TestPoint:TestPoint_Pad_D1.5mm
- TP?: renamed from TP17; footprint (none) -> TestPoint:TestPoint_Pad_D1.5mm
- TP?: renamed from TP15; footprint (none) -> TestPoint:TestPoint_Pad_D1.5mm
- TP?: renamed from TP14; footprint (none) -> TestPoint:TestPoint_Pad_D1.5mm
- U?: renamed from U6; footprint (none) -> Package_TO_SOT_SMD:SOT-23-5
- U?: renamed from U7; footprint (none) -> Package_SO:SOIC-8-1EP_3.9x4.9mm_P1.27mm_EP2.29x3mm_ThermalVias
- U?: renamed from U9; footprint (none) -> Package_TO_SOT_SMD:SOT-353_SC-70-5_Handsoldering
- U?: renamed from U8; footprint Relay_THT:Relay_DPDT_AXICOM_IMSeries_Pitch5.08mm -> Package_TO_SOT_SMD:SOT-23-6_Handsoldering
Connections:
- net +3.3V: now also EC?.1
- net +5V: now also EC?.1
- net +6V: now also D?.1, EC?.1, EC?.1; no longer D?.2
- net +BATT: now also EC?.1, EC?.1
- net GND: now also J?.6 (BODY_GND), U?.9 (GND), EC?.2, EC?.2, EC?.2, EC?.2, EC?.2, EC?.2
- net at L?.2, Q?.5 (D), Q?.6 (D)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: now also D?.2; no longer D?.1
- net VBUS: now reaches C?.2, C?.2, J?.1 (VBUS), R?.1, U?.4 (VDD)
- net at R?.1: now also U?.3 (VFB); no longer U?.5 (VFB)
- no-connect marks 3 -> 8

Commit message: doing placement
Parts:
- gave numbers to parts that had none: 56

Commit message: Working on lib and pcb layout
Parts:
- J4: footprint Connector_USB:USB_Micro-AB_Molex_47590-0001 -> _HW_HandyRadio_Footprint:USB_Micro-AB_Molex_47590-0001
- R30: footprint Potentiometer_SMD:Potentiometer_Bourns_TC33X_Vertical -> _HW_HandyRadio_Footprint:Potentiometer_Bourns_TC33X_Vertical
- U5: footprint Package_SO:SOIC-8-1EP_3.9x4.9mm_P1.27mm_EP2.29x3mm_ThermalVias -> _HW_HandyRadio_Footprint:Infineon_PG-DSO-8-27_3.9x4.9mm_EP2.65x3mm_ThermalVias
Changed lines of the file:
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@@
     (effects (font (size 1.27 1.27)) (justify right))
   )
-  (symbol (lib_name "TPC_6") (lib_id "HandyRadio:TPC") (at 393.7 72.39 90) (unit 1)
+  (symbol (lib_id "HandyRadio:TPC") (at 393.7 72.39 90) (unit 1)
     (in_bom yes) (on_board yes) (fields_autoplaced)
     (property "Reference" "TP17" (id 0) (at 396.24 64.7699 90)
@@
     (pin "1")
   )
-  (symbol (lib_name "TPC_1") (lib_id "HandyRadio:TPC") (at 179.07 77.47 90) (unit 1)
+  (symbol (lib_id "HandyRadio:TPC") (at 179.07 77.47 90) (unit 1)
     (in_bom yes) (on_board yes) (fields_autoplaced)
     (property "Reference" "TP11" (id 0) (at 181.61 69.8499 90)
@@
       (effects (font (size 1.27 1.27)) (justify left))
     )
-    (property "Footprint" "Potentiometer_SMD:Potentiometer_Bourns_TC33X_Vertical" (id 2) (at 322.58 147.32 0)
+    (property "Footprint" "_HW_HandyRadio_Footprint:Potentiometer_Bourns_TC33X_Vertical" (id 2) (at 322.58 147.32 0)
       (effects (font (size 1.27 1.27)) hide)
     )
@@
     (pin "2")
   )
-  (symbol (lib_name "TPC_8") (lib_id "HandyRadio:TPC") (at 391.16 191.77 90) (unit 1)
+  (symbol (lib_id "HandyRadio:TPC") (at 391.16 191.77 90) (unit 1)
     (in_bom yes) (on_board yes) (fields_autoplaced)
     (property "Reference" "TP16" (id 0) (at 393.7 184.1499 90)
@@
     (pin "2")
   )
-  (symbol (lib_name "TPC_7") (lib_id "HandyRadio:TPC") (at 397.51 212.09 0) (unit 1)
+  (symbol (lib_id "HandyRadio:TPC") (at 397.51 212.09 0) (unit 1)
     (in_bom yes) (on_board yes) (fields_autoplaced)
     (property "Reference" "TP18" (id 0) (at 406.4 210.8199 0)
@@
     (property "Reference" "J4" (id 0) (at 21.59 72.39 0))
     (property "Value" "USB_uAB_RECEP" (id 1) (at 21.59 74.93 0))
-    (property "Footprint" "Connector_USB:USB_Micro-AB_Molex_47590-0001" (id 2) (at 16.51 69.85 0)
+    (property "Footprint" "_HW_HandyRadio_Footprint:USB_Micro-AB_Molex_47590-0001" (id 2) (at 16.51 69.85 0)
       (effects (font (size 1.27 1.27)) hide)
     )
@@
     (pin "5")
   )
-  (symbol (lib_name "TPC_5") (lib_id "HandyRadio:TPC") (at 406.4 72.39 90) (unit 1)
+  (symbol (lib_id "HandyRadio:TPC") (at 406.4 72.39 90) (unit 1)
     (in_bom yes) (on_board yes) (fields_autoplaced)
     (property "Reference" "TP19" (id 0) (at 408.94 64.7699 90)
@@
     (pin "1")
   )
-  (symbol (lib_name "TPC_4") (lib_id "HandyRadio:TPC") (at 340.36 107.95 0) (unit 1)
+  (symbol (lib_id "HandyRadio:TPC") (at 340.36 107.95 0) (unit 1)
     (in_bom yes) (on_board yes) (fields_autoplaced)
     (property "Reference" "TP15" (id 0) (at 349.25 106.6799 0)
@@
     (pin "1")
   )
-  (symbol (lib_name "TPC_3") (lib_id "HandyRadio:TPC") (at 195.58 212.09 0) (unit 1)
+  (symbol (lib_id "HandyRadio:TPC") (at 195.58 212.09 0) (unit 1)
     (in_bom yes) (on_board yes) (fields_autoplaced)
     (property "Reference" "TP13" (id 0) (at 204.47 210.8199 0)
@@
     (property "Reference" "U5" (id 0) (at 121.92 186.69 0))
     (property "Value" "AP7361EA" (id 1) (at 121.92 189.23 0))
-    (property "Footprint" "Package_SO:SOIC-8-1EP_3.9x4.9mm_P1.27mm_EP2.29x3mm_ThermalVias" (id 2) (at 124.46 185.42 0)
+    (property "Footprint" "_HW_HandyRadio_Footprint:Infineon_PG-DSO-8-27_3.9x4.9mm_EP2.65x3mm_ThermalVias" (id 2) (at 124.46 185.42 0)
       (effects (font (size 1.27 1.27)) hide)
     )
@@
     (pin "2")
   )
-  (symbol (lib_name "TPC_2") (lib_id "HandyRadio:TPC") (at 191.77 193.04 90) (unit 1)
+  (symbol (lib_id "HandyRadio:TPC") (at 191.77 193.04 90) (unit 1)
     (in_bom yes) (on_board yes) (fields_autoplaced)
     (property "Reference" "TP12" (id 0) (at 194.31 185.4199 90)

Commit message: serious modification has been done
Parts:
- removed EC11, EC7: 4u7F/6.3V, Capacitor_Tantalum_SMD:CP_EIA-2012-12_Kemet-R_Pad1.30x1.05mm_HandSolder, symbol HandyRadio:4u7F/6.3V
- removed EC9: 2u2F/10V, Capacitor_Tantalum_SMD:CP_EIA-2012-12_Kemet-R_Pad1.30x1.05mm_HandSolder, symbol HandyRadio:2u2F{brace}slash}10V
- removed R23: 2KR, Resistor_SMD:R_0805_2012Metric_Pad1.20x1.40mm_HandSolder, symbol HandyRadio:2KR
- added C41, C42, C45, C46, C47, C48: 1uF, Capacitor_SMD:C_0805_2012Metric_Pad1.18x1.45mm_HandSolder, symbol HandyRadio:1uF
- added R20: 2KR, Resistor_SMD:R_0805_2012Metric_Pad1.20x1.40mm_HandSolder, symbol HandyRadio:2KR
- added R22, R23: 10KR, Resistor_SMD:R_0805_2012Metric_Pad1.20x1.40mm_HandSolder, symbol HandyRadio:10KR
- renumbered C22 to C24, C23 to C25, C24 to C26, C25 to C27, C26 to C28, C27 to C29, C28 to C30, C29 to C31, C30 to C32, C31 to C33, C32 to C34, C33 to C35, C34 to C36, C35 to C37, C36 to C38, C37 to C39, C38 to C40, C39 to C43, C40 to C44, C42 to C49, C41 to C50, C43 to C51, D3 to D2, EC8 to EC1, EC10 to EC2, EC12 to EC3, R24 to R21, R25 to R24, R26 to R25, R27 to R26, R28 to R27, R29 to R28, R30 to R29, R31 to R30, R32 to R31, TP17 to TP16, TP16 to TP17
Connections:
- net +3.3V: now also C45.2, C46.2, C47.2, C48.2
- net +5V: now also C41.2, C42.2
- net +BATT: now also R22.2
- net BATT_STAT: now also R22.1, R23.2
- net GND: now also J4.1 (GND), C41.1, C42.1, C45.1, C46.1, C47.1, C48.1, R20.1, R23.1; no longer J4.5 (GND)
- net VBUS: now also J4.5 (VBUS); no longer J4.1 (VBUS)
- net PROG: now reaches U4.5 (PROG)
- net PROG: now also R20.2
- net LDO3V3_EN: now reaches R26.2, U7.3 (EN)
Other:
- moved on the sheet: C31, C43, C50, R26, TP13, TP17, TP18, U7

Commit message: layout is in progress
Connections:
- net L_O: now reaches D2.2, L1.2, Q1.5 (D), Q1.6 (D), Q1.7 (D), Q1.8 (D)
- net +3.3V renamed +3V3
Changed lines of the file:
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@@
     (effects (font (size 3 3)) (justify left bottom))
+  )
+  (label "L_O" (at 273.05 80.01 0)
+    (effects (font (size 1.27 1.27)) (justify left bottom))
   )
   (label "DELAY" (at 242.57 105.41 0)
@@
     (pin "1")
   )
+  (symbol (lib_id "power:+3V3") (at 405.13 194.31 270) (unit 1)
+    (in_bom yes) (on_board yes) (fields_autoplaced)
+    (property "Reference" "#PWR?" (id 0) (at 401.32 194.31 0)
+      (effects (font (size 1.27 1.27)) hide)
+    )
+    (property "Value" "+3V3" (id 1) (at 408.94 194.3099 90)
+      (effects (font (size 1.27 1.27)) (justify left))
+    )
+    (property "Footprint" "" (id 2) (at 405.13 194.31 0)
+      (effects (font (size 1.27 1.27)) hide)
+    )
+    (property "Datasheet" "" (id 3) (at 405.13 194.31 0)
+      (effects (font (size 1.27 1.27)) hide)
+    )
+    (pin "1")
+  )
   (symbol (lib_id "HandyRadio:TPC") (at 398.78 191.77 90) (unit 1)
     (in_bom yes) (on_board yes) (fields_autoplaced)
@@
       (effects (font (size 1.27 1.27)) hide)
     )
-    (pin "1")
-  )
-  (symbol (lib_id "power:+3.3V") (at 405.13 194.31 270) (unit 1)
-    (in_bom yes) (on_board yes) (fields_autoplaced)
-    (property "Reference" "#PWR049" (id 0) (at 401.32 194.31 0)
-      (effects (font (size 1.27 1.27)) hide)
-    )
-    (property "Value" "+3.3V" (id 1) (at 408.94 194.3099 90)
-      (effects (font (size 1.27 1.27)) (justify left))
-    )
-    (property "Footprint" "" (id 2) (at 405.13 194.31 0)
-      (effects (font (size 1.27 1.27)) hide)
-    )
-    (property "Datasheet" "" (id 3) (at 405.13 194.31 0)
-      (effects (font (size 1.27 1.27)) hide)
-    )

Commit message: some modification
Parts:
- removed R31: 16KR5, Resistor_SMD:R_0805_2012Metric_Pad1.20x1.40mm_HandSolder, symbol HandyRadio:16KR5
- added R512: 16K5R, Resistor_SMD:R_0805_2012Metric_Pad1.20x1.40mm_HandSolder, symbol HandyRadio:16K5R
- renumbered C24 to C501, C25 to C502, C26 to C503, C27 to C504, C28 to C505, C29 to C506, C30 to C507, C31 to C508, C32 to C509, C33 to C510, C34 to C511, C35 to C512, C36 to C513, C37 to C514, C38 to C515, C39 to C516, C40 to C517, C41 to C518, C42 to C519, C43 to C520, C44 to C521, C45 to C522, C46 to C523, C47 to C524, C48 to C525, C49 to C526, C50 to C527, C51 to C528, D2 to D501, EC1 to EC501, EC2 to EC502, EC3 to EC503, J4 to J501, J5 to J502, L1 to L501, Q1 to Q501, R20 to R501, R21 to R502, R22 to R503, R23 to R504, R24 to R505, R25 to R506, R26 to R507, R27 to R508, R28 to R509, R29 to R510, R30 to R511, TP11 to TP501, TP12 to TP502, TP13 to TP503, TP14 to TP504, TP15 to TP505, TP16 to TP506, TP17 to TP507, TP18 to TP508, TP19 to TP509, U4 to U501, U5 to U502, U6 to U503, U7 to U504
Connections:
- net GND: now also R512.1
- net at C521.1, R506.2, R508.2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: now also R512.2
