File: HandyRadio/HW/V1_09302022/1- Design Files/_HW_HandyRadio_/[06] - DCDC PWS.kicad_sch (KiCad schematic)
At the start: 61 parts, among them J501 USB_uAB_RECEP, J502 XH_CONN_2POS_R/A, Q501 IRF7401TRPBF, U501 MCP73831, U502 AP7361EA, U503 R1211N002B, U504 MIC5365-3.3

Commit message: routing on progress
Parts:
- TC502: renamed from EC502; value 2u2F/10V -> 2u2F/10V; symbol HandyRadio:2u2F{brace}slash}10V -> HandyRadio:2u2F/10V
- TC503: renamed from EC503; value 2u2F/10V -> 2u2F/10V; symbol HandyRadio:2u2F{brace}slash}10V -> HandyRadio:2u2F/10V
- renumbered EC501 to TC501
Changed lines of the file:
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@@
   (symbol (lib_id "HandyRadio:4u7F{slash}6.3V") (at 204.47 106.68 270) (unit 1)
     (in_bom yes) (on_board yes) (fields_autoplaced)
-    (property "Reference" "EC501" (id 0) (at 208.28 112.6489 90)
+    (property "Reference" "TC501" (id 0) (at 208.28 112.6489 90)
       (effects (font (size 1.27 1.27)) (justify left))
     )
@@
     (pin "2")
   )
-  (symbol (lib_id "HandyRadio:2u2F{brace}slash}10V") (at 375.92 99.06 270) (unit 1)
-    (in_bom yes) (on_board yes) (fields_autoplaced)
-    (property "Reference" "EC503" (id 0) (at 379.73 105.0289 90)
-      (effects (font (size 1.27 1.27)) (justify left))
-    )
-    (property "Value" "2u2F{slash}10V" (id 1) (at 379.73 107.5689 90)
-      (effects (font (size 1.27 1.27)) (justify left))
-    )
+  (symbol (lib_id "HandyRadio:2u2F{slash}10V") (at 375.92 99.06 270) (unit 1)
+    (in_bom yes) (on_board yes)
+    (property "Reference" "TC503" (id 0) (at 381 105.41 90))
+    (property "Value" "2u2F/10V" (id 1) (at 383.54 107.95 90))
     (property "Footprint" "Capacitor_Tantalum_SMD:CP_EIA-2012-12_Kemet-R_Pad1.30x1.05mm_HandSolder" (id 2) (at 383.54 105.41 0)
       (effects (font (size 1.27 1.27)) hide)
@@
     (pin "2")
   )
-  (symbol (lib_id "HandyRadio:2u2F{brace}slash}10V") (at 358.14 99.06 270) (unit 1)
-    (in_bom yes) (on_board yes) (fields_autoplaced)
-    (property "Reference" "EC502" (id 0) (at 361.95 105.0289 90)
-      (effects (font (size 1.27 1.27)) (justify left))
-    )
-    (property "Value" "2u2F{slash}10V" (id 1) (at 361.95 107.5689 90)
-      (effects (font (size 1.27 1.27)) (justify left))
-    )
+  (symbol (lib_id "HandyRadio:2u2F{slash}10V") (at 358.14 99.06 270) (unit 1)
+    (in_bom yes) (on_board yes)
+    (property "Reference" "TC502" (id 0) (at 363.22 105.41 90))
+    (property "Value" "2u2F/10V" (id 1) (at 365.76 107.95 90))
     (property "Footprint" "Capacitor_Tantalum_SMD:CP_EIA-2012-12_Kemet-R_Pad1.30x1.05mm_HandSolder" (id 2) (at 365.76 105.41 0)
       (effects (font (size 1.27 1.27)) hide)

Commit message: Ready to release the HW :smile:
Other:
- note added: "CHECKED"
- moved on the sheet: C501, C503, C505, C507, C508
