File: HandyRadio/HW/V1_09302022/1- Design Files/_HW_HandyRadio_/[03] - MCU, RTC, OLED, PB, LED.kicad_sch (KiCad schematic)
At the start: 0 parts

Commit message: 1/6 of the hardware has been done
Parts:
- added C? (x2): 10nF, symbol HandyRadio:10nF
- added C? (x4): 4u7F, symbol HandyRadio:4u7F
- added C? (x8): 100nF, symbol HandyRadio:100nF
- added D?: LED_R, symbol HandyRadio:LED_R
- added J?: MHDR_4POS_1ROW, symbol HandyRadio:MHDR_4POS_1ROW
- added J?: RECEP_6POS_1ROW, symbol HandyRadio:RECEP_6POS_1ROW
- added R? (x6): 10KR, symbol HandyRadio:10KR
- added R? (x3): 1KR, symbol HandyRadio:1KR
- added SW? (x3): SPST_NO_RA, symbol HandyRadio:SPST_NO_RA
- added U?: IR_REC_38KHz, symbol HandyRadio:IR_REC_38KHz
- added U?: STM32F030F4P6, symbol HandyRadio:STM32F030F4P6
Connections:
- new net: D?.2, R?.2
- new net: C?.2, R?.2, SW?.2, U?.6 (PA0)
- new net: C?.2, R?.2, SW?.2, U?.7 (PA1)
- new net: J?.4, R?.1
- new net: C?.2, R?.2, SW?.2, U?.8 (PA2)
- new net +3V3: C?.2, C?.2, C?.2, C?.2, C?.2, C?.2, C?.2, C?.2, C?.2, C?.2, D?.1, J?.5, R?.2, R?.2, SW?.1, SW?.1, SW?.1, U?.16 (VDD), U?.3 (VCC), U?.5 (VDDA)
- new net BEEP_OUPUT: R?.1, U?.10 (PA4)
- new net BEEP_OUTPUT: R?.2
- new net GND: C?.1, C?.1, C?.1, C?.1, C?.1, C?.1, C?.1, C?.1, C?.1, C?.1, C?.1, C?.1, C?.1, C?.1, J?.1, J?.6, R?.1, R?.1, R?.1, R?.1, U?.15 (VSS), U?.2 (GND)
- new net I2C_SCL: J?.4, U?.17 (PA9)
- new net I2C_SDA: J?.3, U?.18 (PA10)
- new net IR_INPUT: U?.1 (OUTPUT), U?.12 (PA6)
- new net LED_IND: R?.1, U?.14 (PB1)
- new net MCU_BOOT0: R?.2, U?.1 (BOOT0)
- new net MCU_NRST: C?.2, R?.1, U?.4 (NRST)
- new net OLED_RST: J?.2, R?.2
- new net SWCLK: J?.2, U?.20 (PA14)
- new net SWDIO: J?.3, R?.1, U?.19 (PA13)
- no-connect marks 0 -> 3
Other:
- note added: "1- DC --> DC 2- RES --> RST 3- D1 --> SDA 4- D0 --> SCL 5- VCC --> +3V3 6- GND --> GROUND"
- note added: "INFO:"
- note added: "PROGRAMMER PINS"

Commit message: 2/6 HandyRadio HW has been done
Connections:
- net BEEP_OUTPUT renamed BEEP_SIG
Changed lines of the file:
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@@
     (effects (font (size 1.27 1.27)) (justify left))
   )
-  (hierarchical_label "BEEP_OUTPUT" (shape output) (at 262.89 93.98 0)
+  (hierarchical_label "BEEP_SIG" (shape output) (at 262.89 93.98 0)
     (effects (font (size 1.27 1.27)) (justify left))
   )
@@
     (pin "2")
   )
-  (symbol (lib_id "HandyRadio:100nF") (at 36.83 118.11 90) (unit 1)
+  (symbol (lib_name "100nF_2") (lib_id "HandyRadio:100nF") (at 36.83 118.11 90) (unit 1)
     (in_bom yes) (on_board yes) (fields_autoplaced)
     (property "Reference" "C?" (id 0) (at 40.64 109.2199 90)
@@
     (pin "2")
   )
-  (symbol (lib_id "HandyRadio:100nF") (at 341.63 107.95 90) (unit 1)
+  (symbol (lib_name "100nF_6") (lib_id "HandyRadio:100nF") (at 341.63 107.95 90) (unit 1)
     (in_bom yes) (on_board yes) (fields_autoplaced)
     (property "Reference" "C?" (id 0) (at 345.44 99.0599 90)
@@
     (pin "3")
   )
-  (symbol (lib_id "HandyRadio:100nF") (at 367.03 107.95 90) (unit 1)
+  (symbol (lib_name "100nF_5") (lib_id "HandyRadio:100nF") (at 367.03 107.95 90) (unit 1)
     (in_bom yes) (on_board yes) (fields_autoplaced)
     (property "Reference" "C?" (id 0) (at 370.84 99.0599 90)
@@
     (pin "1")
   )
-  (symbol (lib_id "HandyRadio:10KR") (at 354.33 107.95 90) (unit 1)
+  (symbol (lib_name "10KR_5") (lib_id "HandyRadio:10KR") (at 354.33 107.95 90) (unit 1)
     (in_bom yes) (on_board yes) (fields_autoplaced)
     (property "Reference" "R?" (id 0) (at 356.87 99.0599 90)
@@
     (pin "2")
   )
-  (symbol (lib_id "HandyRadio:100nF") (at 74.93 129.54 90) (unit 1)
+  (symbol (lib_name "100nF_3") (lib_id "HandyRadio:100nF") (at 74.93 129.54 90) (unit 1)
     (in_bom yes) (on_board yes) (fields_autoplaced)
     (property "Reference" "C?" (id 0) (at 78.74 120.6499 90)
@@
     (pin "1")
   )
-  (symbol (lib_id "HandyRadio:10KR") (at 379.73 107.95 90) (unit 1)
+  (symbol (lib_name "10KR_4") (lib_id "HandyRadio:10KR") (at 379.73 107.95 90) (unit 1)
     (in_bom yes) (on_board yes) (fields_autoplaced)
     (property "Reference" "R?" (id 0) (at 382.27 99.0599 90)
@@
     (pin "2")
   )
-  (symbol (lib_id "HandyRadio:100nF") (at 316.23 107.95 90) (unit 1)
+  (symbol (lib_name "100nF_7") (lib_id "HandyRadio:100nF") (at 316.23 107.95 90) (unit 1)
     (in_bom yes) (on_board yes) (fields_autoplaced)
     (property "Reference" "C?" (id 0) (at 320.04 99.0599 90)
@@
     (pin "2")
   )
-  (symbol (lib_id "HandyRadio:100nF") (at 356.87 185.42 90) (unit 1)
+  (symbol (lib_name "100nF_4") (lib_id "HandyRadio:100nF") (at 356.87 185.42 90) (unit 1)
     (in_bom yes) (on_board yes) (fields_autoplaced)
     (property "Reference" "C?" (id 0) (at 360.68 176.5299 90)

Commit message: Schematic is almost done
Changed lines of the file:
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@@
     (effects (font (size 1.27 1.27)) (justify left bottom))
   )
-  (hierarchical_label "I2C_SCL" (shape output) (at 262.89 106.68 0)
+  (hierarchical_label "I2C_SCL" (shape bidirectional) (at 262.89 106.68 0)
     (effects (font (size 1.27 1.27)) (justify left))
   )

Commit message: Schematic is almost Done
Parts:
- removed C?: 4u7F, symbol HandyRadio:4u7F
- added C? (x5): 10uF, symbol HandyRadio:10uF
- added R?: 10KR, symbol HandyRadio:10KR
- added R?: 47R, symbol HandyRadio:47R
- added TP? (x9): TPC, symbol HandyRadio:TPC
Connections:
- net +3V3: now also C?.2, C?.2, C?.2, C?.2, C?.2, R?.1, R?.2; no longer C?.2, U?.3 (VCC)
- net GND: now also C?.1, C?.1, C?.1, C?.1, C?.1, TP?.1, TP?.1, TP?.1, TP?.1
- net I2C_SCL: now also TP?.1
- net I2C_SDA: now also TP?.1
- net IR_INPUT: now also R?.1, TP?.1
- net MCU_NRST: now also TP?.1
- net BATT_STAT: now reaches U?.13 (PA7)
- net BATT_STAT: now also TP?.1
- net FM/SW_SEL: now reaches U?.9 (PA3)
- new net: C?.2, R?.2, U?.3 (VCC)
Other:
- note added: "LAYOUT:"
- note added: "RC Filter should be connected closely between Vcc pin and GND pin."
- company: (none) -> Siavash Taher Parvar
- title: (none) -> Handy Radio
- moved on the sheet: C?, D?, J?, R?, SW?, U?

Commit message: 95 SCHEMATIC HAS BEEN DONE
Parts:
- gave numbers to parts that had none: 46

Commit message: Schematic has been double checked
Parts:
- removed TP4: TPC, symbol HandyRadio:TPC
- added R?: 47R, symbol HandyRadio:47R
- added R? (x2): 10KR, symbol HandyRadio:10KR
- added TP? (x2): TPC, symbol HandyRadio:TPC
Connections:
- net +3V3: now also R?.2, R?.2; no longer D1.1
- net BATT_STAT: now also U1.11 (PA5), TP?.1; no longer U1.13 (PA7)
- net I2C_SCL: now also R?.1
- net I2C_SDA: now also R?.1
- net PB_1: now reaches C18.2, R11.2, SW3.2, U1.6 (PA0)
- net PB_2: now reaches C13.2, R10.2, SW2.2, U1.7 (PA1)
- net PB_3: now reaches C10.2, R8.2, SW1.2, U1.8 (PA2)
- new net +3.3V: D1.1
- new net SI47_CLK: R?.1, R?.2, TP?.1, U1.13 (PA7)
Other:
- note added: "DNF"
- note added: "TP List TP1 = MCU_RESET TP2 = GND TP3 = IR_RECEIVER TP4 = BATT_STAT TP5 = I2C_SCL TP6 = I2C_SDA TP7 = GND TP8 = GND TP9 = GND"
- moved on the sheet: C1, C10, C11, C12, C13, C14, C15, C16, C17, C18, C2, C3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

Commit message: 99% SCHEMATIC HAS BEEN DONE
Parts:
- gave numbers to parts that had none: 5
- renumbered R7 to R10, R8 to R11, R9 to R12, R10 to R13, R11 to R14, R5 to R6, R6 to R9, TP3 to TP10
Changed lines of the file:
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@@
   (symbol (lib_id "HandyRadio:10KR") (at 297.18 120.65 90) (unit 1)
     (in_bom yes) (on_board yes) (fields_autoplaced)
-    (property "Reference" "R6" (id 0) (at 299.72 111.7599 90)
+    (property "Reference" "R9" (id 0) (at 299.72 111.7599 90)
       (effects (font (size 1.27 1.27)) (justify right))
     )
@@
   (symbol (lib_id "power:GND") (at 284.48 147.32 0) (unit 1)
     (in_bom yes) (on_board yes) (fields_autoplaced)
-    (property "Reference" "#PWR011" (id 0) (at 284.48 153.67 0)
+    (property "Reference" "#PWR012" (id 0) (at 284.48 153.67 0)
       (effects (font (size 1.27 1.27)) hide)
     )
@@
   (symbol (lib_id "HandyRadio:47R") (at 207.01 97.79 0) (unit 1)
     (in_bom yes) (on_board yes)
-    (property "Reference" "R?" (id 0) (at 223.52 96.52 0))
+    (property "Reference" "R5" (id 0) (at 223.52 96.52 0))
     (property "Value" "47R" (id 1) (at 204.47 96.52 0))
     (property "Footprint" "" (id 2) (at 209.55 92.71 0)
@@
   (symbol (lib_id "power:GND") (at 370.84 109.22 0) (unit 1)
     (in_bom yes) (on_board yes) (fields_autoplaced)
-    (property "Reference" "#PWR023" (id 0) (at 370.84 115.57 0)
+    (property "Reference" "#PWR024" (id 0) (at 370.84 115.57 0)
       (effects (font (size 1.27 1.27)) hide)
     )
@@
   (symbol (lib_id "power:GND") (at 341.63 189.23 0) (unit 1)
     (in_bom yes) (on_board yes) (fields_autoplaced)
-    (property "Reference" "#PWR017" (id 0) (at 341.63 195.58 0)
+    (property "Reference" "#PWR018" (id 0) (at 341.63 195.58 0)
       (effects (font (size 1.27 1.27)) hide)
     )
@@
   (symbol (lib_id "power:+3V3") (at 351.79 60.96 0) (unit 1)
     (in_bom yes) (on_board yes) (fields_autoplaced)
-    (property "Reference" "#PWR019" (id 0) (at 351.79 64.77 0)
+    (property "Reference" "#PWR020" (id 0) (at 351.79 64.77 0)
       (effects (font (size 1.27 1.27)) hide)
     )
@@
   (symbol (lib_name "10KR_5") (lib_id "HandyRadio:10KR") (at 351.79 104.14 90) (unit 1)
     (in_bom yes) (on_board yes) (fields_autoplaced)
-    (property "Reference" "R10" (id 0) (at 354.33 95.2499 90)
+    (property "Reference" "R13" (id 0) (at 354.33 95.2499 90)
       (effects (font (size 1.27 1.27)) (justify right))
     )
@@
   (symbol (lib_name "10KR_4") (lib_id "HandyRadio:10KR") (at 377.19 104.14 90) (unit 1)
     (in_bom yes) (on_board yes) (fields_autoplaced)
-    (property "Reference" "R11" (id 0) (at 379.73 95.2499 90)
+    (property "Reference" "R14" (id 0) (at 379.73 95.2499 90)
       (effects (font (size 1.27 1.27)) (justify right))
     )
@@
   (symbol (lib_id "power:+3V3") (at 261.62 143.51 0) (unit 1)
     (in_bom yes) (on_board yes) (fields_autoplaced)
-    (property "Reference" "#PWR?" (id 0) (at 261.62 147.32 0)
+    (property "Reference" "#PWR011" (id 0) (at 261.62 147.32 0)
       (effects (font (size 1.27 1.27)) hide)
     )
@@
   (symbol (lib_id "HandyRadio:TPC") (at 287.02 95.25 0) (unit 1)
     (in_bom yes) (on_board yes) (fields_autoplaced)
-    (property "Reference" "TP3" (id 0) (at 295.91 93.9799 0)
+    (property "Reference" "TP10" (id 0) (at 295.91 93.9799 0)
       (effects (font (size 1.27 1.27)) (justify left))
     )
@@
   (symbol (lib_id "HandyRadio:TPC") (at 264.16 91.44 0) (unit 1)
     (in_bom yes) (on_board yes) (fields_autoplaced)
-    (property "Reference" "TP?" (id 0) (at 273.05 90.1699 0)
+    (property "Reference" "TP4" (id 0) (at 273.05 90.1699 0)
       (effects (font (size 1.27 1.27)) (justify left))
     )
@@
   (symbol (lib_id "power:GND") (at 365.76 189.23 0) (unit 1)
     (in_bom yes) (on_board yes) (fields_autoplaced)
-    (property "Reference" "#PWR021" (id 0) (at 365.76 195.58 0)
+    (property "Reference" "#PWR022" (id 0) (at 365.76 195.58 0)
       (effects (font (size 1.27 1.27)) hide)
     )
@@
   (symbol (lib_id "HandyRadio:10KR") (at 326.39 104.14 90) (unit 1)
     (in_bom yes) (on_board yes) (fields_autoplaced)
-    (property "Reference" "R8" (id 0) (at 328.93 95.2499 90)
+    (property "Reference" "R11" (id 0) (at 328.93 95.2499 90)
       (effects (font (size 1.27 1.27)) (justify right))
     )
@@
   (symbol (lib_id "power:+3.3V") (at 369.57 207.01 270) (unit 1)
     (in_bom yes) (on_board yes) (fields_autoplaced)
-    (property "Reference" "#PWR?" (id 0) (at 365.76 207.01 0)
+    (property "Reference" "#PWR023" (id 0) (at 365.76 207.01 0)
       (effects (font (size 1.27 1.27)) hide)
     )
@@
   (symbol (lib_id "power:GND") (at 320.04 109.22 0) (unit 1)
     (in_bom yes) (on_board yes) (fields_autoplaced)
-    (property "Reference" "#PWR014" (id 0) (at 320.04 115.57 0)
+    (property "Reference" "#PWR015" (id 0) (at 320.04 115.57 0)
       (effects (font (size 1.27 1.27)) hide)
     )
@@
   (symbol (lib_name "10KR_3") (lib_id "HandyRadio:10KR") (at 207.01 107.95 0) (unit 1)
     (in_bom yes) (on_board yes)
-    (property "Reference" "R5" (id 0) (at 222.25 106.68 0))
+    (property "Reference" "R6" (id 0) (at 222.25 106.68 0))
     (property "Value" "10KR" (id 1) (at 204.47 106.68 0))
     (property "Footprint" "" (id 2) (at 207.01 107.95 0)
@@
   (symbol (lib_id "power:GND") (at 345.44 109.22 0) (unit 1)
     (in_bom yes) (on_board yes) (fields_autoplaced)
-    (property "Reference" "#PWR018" (id 0) (at 345.44 115.57 0)
+    (property "Reference" "#PWR019" (id 0) (at 345.44 115.57 0)
       (effects (font (size 1.27 1.27)) hide)
     )
@@
   (symbol (lib_id "HandyRadio:47R") (at 344.17 127 0) (unit 1)
     (in_bom yes) (on_board yes)
-    (property "Reference" "R9" (id 0) (at 359.41 125.73 0))
+    (property "Reference" "R12" (id 0) (at 359.41 125.73 0))
     (property "Value" "47R" (id 1) (at 342.9 125.73 0))
     (property "Footprint" "" (id 2) (at 346.71 121.92 0)
@@
   (symbol (lib_id "power:+3V3") (at 377.19 60.96 0) (unit 1)
     (in_bom yes) (on_board yes) (fields_autoplaced)
-    (property "Reference" "#PWR024" (id 0) (at 377.19 64.77 0)
+    (property "Reference" "#PWR025" (id 0) (at 377.19 64.77 0)
       (effects (font (size 1.27 1.27)) hide)
     )
@@
   (symbol (lib_id "HandyRadio:10KR") (at 254 161.29 90) (unit 1)
     (in_bom yes) (on_board yes) (fields_autoplaced)
-    (property "Reference" "R?" (id 0) (at 256.54 152.3999 90)
+    (property "Reference" "R7" (id 0) (at 256.54 152.3999 90)
       (effects (font (size 1.27 1.27)) (justify right))
     )
@@
   (symbol (lib_id "power:+3V3") (at 326.39 60.96 0) (unit 1)
     (in_bom yes) (on_board yes) (fields_autoplaced)
-    (property "Reference" "#PWR015" (id 0) (at 326.39 64.77 0)
+    (property "Reference" "#PWR016" (id 0) (at 326.39 64.77 0)
       (effects (font (size 1.27 1.27)) hide)
     )
@@
   (symbol (lib_id "power:+3V3") (at 294.64 127 90) (unit 1)
     (in_bom yes) (on_board yes)
-    (property "Reference" "#PWR012" (id 0) (at 298.45 127 0)
+    (property "Reference" "#PWR013" (id 0) (at 298.45 127 0)
       (effects (font (size 1.27 1.27)) hide)
     )
@@
   (symbol (lib_id "power:+3V3") (at 337.82 170.18 90) (unit 1)
     (in_bom yes) (on_board yes) (fields_autoplaced)
-    (property "Reference" "#PWR016" (id 0) (at 341.63 170.18 0)
+    (property "Reference" "#PWR017" (id 0) (at 341.63 170.18 0)
       (effects (font (size 1.27 1.27)) hide)
     )
@@
   (symbol (lib_id "HandyRadio:10KR") (at 269.24 161.29 90) (unit 1)
     (in_bom yes) (on_board yes) (fields_autoplaced)
-    (property "Reference" "R?" (id 0) (at 271.78 152.3999 90)
+    (property "Reference" "R8" (id 0) (at 271.78 152.3999 90)
       (effects (font (size 1.27 1.27)) (justify right))
     )
@@
   (symbol (lib_id "HandyRadio:1KR") (at 322.58 207.01 0) (unit 1)
     (in_bom yes) (on_board yes)
-    (property "Reference" "R7" (id 0) (at 340.36 205.74 0)
+    (property "Reference" "R10" (id 0) (at 340.36 205.74 0)
       (effects (font (size 1.27 1.27)) (justify right))
     )
@@
   (symbol (lib_id "power:GND") (at 354.33 189.23 0) (unit 1)
     (in_bom yes) (on_board yes) (fields_autoplaced)
-    (property "Reference" "#PWR020" (id 0) (at 354.33 195.58 0)
+    (property "Reference" "#PWR021" (id 0) (at 354.33 195.58 0)
       (effects (font (size 1.27 1.27)) hide)
     )
@@
   (symbol (lib_id "HandyRadio:TPC") (at 262.89 100.33 0) (unit 1)
     (in_bom yes) (on_board yes) (fields_autoplaced)
-    (property "Reference" "TP?" (id 0) (at 271.78 99.0599 0)
+    (property "Reference" "TP3" (id 0) (at 271.78 99.0599 0)
       (effects (font (size 1.27 1.27)) (justify left))
     )
@@
   (symbol (lib_id "power:+3V3") (at 297.18 104.14 0) (unit 1)
     (in_bom yes) (on_board yes) (fields_autoplaced)
-    (property "Reference" "#PWR013" (id 0) (at 297.18 107.95 0)
-      (effects (font (size 1.27 1.27)) hide)
-    )
+    (property "Reference" "#PWR014" (id 0) (at 297.18 107.95 0)
+      (effects (font (size 1.27 1.27)) hide)
+    )

Commit message: almost ready for routing and finishing PCB :D
Parts:
- C?: renamed from C7; footprint (none) -> Capacitor_SMD:C_0805_2012Metric_Pad1.18x1.45mm_HandSolder
- C?: renamed from C1; footprint (none) -> Capacitor_SMD:C_0805_2012Metric_Pad1.18x1.45mm_HandSolder
- C?: renamed from C12; footprint (none) -> Capacitor_SMD:C_0805_2012Metric_Pad1.18x1.45mm_HandSolder
- C?: renamed from C14; footprint (none) -> Capacitor_SMD:C_0805_2012Metric_Pad1.18x1.45mm_HandSolder
- C?: renamed from C17; footprint (none) -> Capacitor_SMD:C_0805_2012Metric_Pad1.18x1.45mm_HandSolder
- C?: renamed from C13; footprint (none) -> Capacitor_SMD:C_0805_2012Metric_Pad1.18x1.45mm_HandSolder
- C?: renamed from C9; footprint (none) -> Capacitor_SMD:C_0805_2012Metric_Pad1.18x1.45mm_HandSolder
- C?: renamed from C5; footprint (none) -> Capacitor_SMD:C_0805_2012Metric_Pad1.18x1.45mm_HandSolder
- C?: renamed from C2; footprint (none) -> Capacitor_SMD:C_0805_2012Metric_Pad1.18x1.45mm_HandSolder
- C?: renamed from C18; footprint (none) -> Capacitor_SMD:C_0805_2012Metric_Pad1.18x1.45mm_HandSolder
- C?: renamed from C8; footprint (none) -> Capacitor_SMD:C_0805_2012Metric_Pad1.18x1.45mm_HandSolder
- C?: renamed from C3; footprint (none) -> Capacitor_SMD:C_0805_2012Metric_Pad1.18x1.45mm_HandSolder
- C?: renamed from C11; footprint (none) -> Capacitor_SMD:C_0805_2012Metric_Pad1.18x1.45mm_HandSolder
- C?: renamed from C10; footprint (none) -> Capacitor_SMD:C_0805_2012Metric_Pad1.18x1.45mm_HandSolder
- C?: renamed from C15; footprint (none) -> Capacitor_SMD:C_0805_2012Metric_Pad1.18x1.45mm_HandSolder
- C?: renamed from C4; footprint (none) -> Capacitor_SMD:C_0805_2012Metric_Pad1.18x1.45mm_HandSolder
- C?: renamed from C16; footprint (none) -> Capacitor_SMD:C_0805_2012Metric_Pad1.18x1.45mm_HandSolder
- C?: renamed from C6; footprint (none) -> Capacitor_SMD:C_0805_2012Metric_Pad1.18x1.45mm_HandSolder
- D?: renamed from D1; footprint (none) -> LED_THT:LED_D5.0mm
- J?: renamed from J1; footprint (none) -> Connector_PinHeader_2.54mm:PinHeader_1x04_P2.54mm_Vertical
- J?: renamed from J2; footprint (none) -> Connector_PinHeader_2.54mm:PinHeader_1x06_P2.54mm_Vertical
- R?: renamed from R9; footprint (none) -> Resistor_SMD:R_0805_2012Metric_Pad1.20x1.40mm_HandSolder
- R?: renamed from R5; footprint (none) -> Resistor_SMD:R_0805_2012Metric_Pad1.20x1.40mm_HandSolder
- R?: renamed from R1; footprint (none) -> Resistor_SMD:R_0805_2012Metric_Pad1.20x1.40mm_HandSolder
- R?: renamed from R13; footprint (none) -> Resistor_SMD:R_0805_2012Metric_Pad1.20x1.40mm_HandSolder
- R?: renamed from R14; footprint (none) -> Resistor_SMD:R_0805_2012Metric_Pad1.20x1.40mm_HandSolder
- R?: renamed from R11; footprint (none) -> Resistor_SMD:R_0805_2012Metric_Pad1.20x1.40mm_HandSolder
- R?: renamed from R6; footprint (none) -> Resistor_SMD:R_0805_2012Metric_Pad1.20x1.40mm_HandSolder
- R?: renamed from R4; footprint (none) -> Resistor_SMD:R_0805_2012Metric_Pad1.20x1.40mm_HandSolder
- R?: renamed from R12; footprint (none) -> Resistor_SMD:R_0805_2012Metric_Pad1.20x1.40mm_HandSolder
- R?: renamed from R7; footprint (none) -> Resistor_SMD:R_0805_2012Metric_Pad1.20x1.40mm_HandSolder
- R?: renamed from R8; footprint (none) -> Resistor_SMD:R_0805_2012Metric_Pad1.20x1.40mm_HandSolder
- R?: renamed from R10; footprint (none) -> Resistor_SMD:R_0805_2012Metric_Pad1.20x1.40mm_HandSolder
- R?: renamed from R2; footprint (none) -> Resistor_SMD:R_0805_2012Metric_Pad1.20x1.40mm_HandSolder
- R?: renamed from R3; footprint (none) -> Resistor_SMD:R_0805_2012Metric_Pad1.20x1.40mm_HandSolder
- SW?: renamed from SW3; footprint (none) -> Button_Switch_THT:SW_Tactile_SKHH_Angled
- SW?: renamed from SW2; footprint (none) -> Button_Switch_THT:SW_Tactile_SKHH_Angled
- SW?: renamed from SW1; footprint (none) -> Button_Switch_THT:SW_Tactile_SKHH_Angled
- TP?: renamed from TP8; footprint (none) -> TestPoint:TestPoint_Pad_D1.5mm
- TP?: renamed from TP5; footprint (none) -> TestPoint:TestPoint_Pad_D1.5mm
- TP?: renamed from TP10; footprint (none) -> TestPoint:TestPoint_Pad_D1.5mm
- TP?: renamed from TP9; footprint (none) -> TestPoint:TestPoint_Pad_D1.5mm
- TP?: renamed from TP4; footprint (none) -> TestPoint:TestPoint_Pad_D1.5mm
- TP?: renamed from TP7; footprint (none) -> TestPoint:TestPoint_Pad_D1.5mm
- TP?: renamed from TP6; footprint (none) -> TestPoint:TestPoint_Pad_D1.5mm
- TP?: renamed from TP2; footprint (none) -> TestPoint:TestPoint_Pad_D1.5mm
- TP?: renamed from TP1; footprint (none) -> TestPoint:TestPoint_Pad_D1.5mm
- TP?: renamed from TP3; footprint (none) -> TestPoint:TestPoint_Pad_D1.5mm
- U?: renamed from U2; footprint (none) -> Connector_PinHeader_2.54mm:PinHeader_1x03_P2.54mm_Vertical
- U?: renamed from U1; footprint (none) -> Package_SO:SSOP-20_4.4x6.5mm_P0.65mm
Connections:
- net +3.3V: now also D?.2; no longer D?.1
- net at R?.2: now also D?.1; no longer D?.2
- net FM/SW_SEL renamed ~{FM}/SW_SEL
