File: HandyRadio/HW/V1_09302022/1- Design Files/_HW_HandyRadio_/[03] - MCU, RTC, OLED, PB, LED.kicad_sch (KiCad schematic)
At the start: 50 parts

Commit message: doing placement
Parts:
- gave numbers to parts that had none: 50

Commit message: Working on lib and pcb layout
Parts:
- SW1, SW2, SW3: footprint Button_Switch_THT:SW_Tactile_SKHH_Angled -> _HW_HandyRadio_Footprint:SW_Tact_SKHH_Angled
Changed lines of the file:
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@@
       (effects (font (size 1.27 1.27)) (justify left))
     )
-    (property "Footprint" "Button_Switch_THT:SW_Tactile_SKHH_Angled" (id 2) (at 388.62 66.04 0)
+    (property "Footprint" "_HW_HandyRadio_Footprint:SW_Tact_SKHH_Angled" (id 2) (at 388.62 66.04 0)
       (effects (font (size 1.27 1.27)) hide)
     )
@@
     (pin "2")
   )
-  (symbol (lib_name "TPC_7") (lib_id "HandyRadio:TPC") (at 264.16 128.27 0) (unit 1)
+  (symbol (lib_id "HandyRadio:TPC") (at 264.16 128.27 0) (unit 1)
     (in_bom yes) (on_board yes) (fields_autoplaced)
     (property "Reference" "TP8" (id 0) (at 273.05 126.9999 0)
@@
       (effects (font (size 1.27 1.27)) (justify left))
     )
-    (property "Footprint" "Button_Switch_THT:SW_Tactile_SKHH_Angled" (id 2) (at 363.22 66.04 0)
+    (property "Footprint" "_HW_HandyRadio_Footprint:SW_Tact_SKHH_Angled" (id 2) (at 363.22 66.04 0)
       (effects (font (size 1.27 1.27)) hide)
     )
@@
     (pin "1")
   )
-  (symbol (lib_name "TPC_3") (lib_id "HandyRadio:TPC") (at 264.16 109.22 0) (unit 1)
+  (symbol (lib_id "HandyRadio:TPC") (at 264.16 109.22 0) (unit 1)
     (in_bom yes) (on_board yes) (fields_autoplaced)
     (property "Reference" "TP5" (id 0) (at 273.05 107.9499 0)
@@
     (pin "2")
   )
-  (symbol (lib_name "TPC_1") (lib_id "HandyRadio:TPC") (at 287.02 95.25 0) (unit 1)
+  (symbol (lib_id "HandyRadio:TPC") (at 287.02 95.25 0) (unit 1)
     (in_bom yes) (on_board yes) (fields_autoplaced)
     (property "Reference" "TP10" (id 0) (at 295.91 93.9799 0)
@@
     (pin "1")
   )
-  (symbol (lib_name "TPC_8") (lib_id "HandyRadio:TPC") (at 264.16 134.62 0) (unit 1)
+  (symbol (lib_id "HandyRadio:TPC") (at 264.16 134.62 0) (unit 1)
     (in_bom yes) (on_board yes) (fields_autoplaced)
     (property "Reference" "TP9" (id 0) (at 273.05 133.3499 0)
@@
     (pin "9")
   )
-  (symbol (lib_name "TPC_5") (lib_id "HandyRadio:TPC") (at 264.16 91.44 0) (unit 1)
+  (symbol (lib_id "HandyRadio:TPC") (at 264.16 91.44 0) (unit 1)
     (in_bom yes) (on_board yes) (fields_autoplaced)
     (property "Reference" "TP4" (id 0) (at 273.05 90.1699 0)
@@
     (pin "1")
   )
-  (symbol (lib_name "TPC_6") (lib_id "HandyRadio:TPC") (at 264.16 121.92 0) (unit 1)
+  (symbol (lib_id "HandyRadio:TPC") (at 264.16 121.92 0) (unit 1)
     (in_bom yes) (on_board yes) (fields_autoplaced)
     (property "Reference" "TP7" (id 0) (at 273.05 120.6499 0)
@@
     (pin "1")
   )
-  (symbol (lib_name "TPC_4") (lib_id "HandyRadio:TPC") (at 264.16 114.3 0) (unit 1)
+  (symbol (lib_id "HandyRadio:TPC") (at 264.16 114.3 0) (unit 1)
     (in_bom yes) (on_board yes) (fields_autoplaced)
     (property "Reference" "TP6" (id 0) (at 273.05 113.0299 0)
@@
     (pin "1")
   )
-  (symbol (lib_name "TPC_9") (lib_id "HandyRadio:TPC") (at 30.48 128.27 180) (unit 1)
+  (symbol (lib_id "HandyRadio:TPC") (at 30.48 128.27 180) (unit 1)
     (in_bom yes) (on_board yes) (fields_autoplaced)
     (property "Reference" "TP2" (id 0) (at 24.13 121.92 0))
@@
       (effects (font (size 1.27 1.27)) (justify left))
     )
-    (property "Footprint" "Button_Switch_THT:SW_Tactile_SKHH_Angled" (id 2) (at 337.82 66.04 0)
+    (property "Footprint" "_HW_HandyRadio_Footprint:SW_Tact_SKHH_Angled" (id 2) (at 337.82 66.04 0)
       (effects (font (size 1.27 1.27)) hide)
     )
@@
     (pin "2")
   )
-  (symbol (lib_name "TPC_2") (lib_id "HandyRadio:TPC") (at 262.89 100.33 0) (unit 1)
+  (symbol (lib_id "HandyRadio:TPC") (at 262.89 100.33 0) (unit 1)
     (in_bom yes) (on_board yes) (fields_autoplaced)
     (property "Reference" "TP3" (id 0) (at 271.78 99.0599 0)

Commit message: serious modification has been done
Parts:
- removed C2: 4u7F, Capacitor_SMD:C_0805_2012Metric_Pad1.18x1.45mm_HandSolder, symbol HandyRadio:4u7F
- removed C3: 100nF, Capacitor_SMD:C_0805_2012Metric_Pad1.18x1.45mm_HandSolder, symbol HandyRadio:100nF
- removed C4: 10nF, Capacitor_SMD:C_0805_2012Metric_Pad1.18x1.45mm_HandSolder, symbol HandyRadio:10nF
- removed R14: 10KR, Resistor_SMD:R_0805_2012Metric_Pad1.20x1.40mm_HandSolder, symbol HandyRadio:10KR
- removed R2: 1KR, Resistor_SMD:R_0805_2012Metric_Pad1.20x1.40mm_HandSolder, symbol HandyRadio:1KR
- removed U1: STM32F030F4P6, Package_SO:SSOP-20_4.4x6.5mm_P0.65mm, symbol HandyRadio:STM32F030F4P6
- added C5: 100nF, Capacitor_SMD:C_0805_2012Metric_Pad1.18x1.45mm_HandSolder, symbol HandyRadio:100nF
- added R12, R15, R16, R9: 10KR, Resistor_SMD:R_0805_2012Metric_Pad1.20x1.40mm_HandSolder, symbol HandyRadio:10KR
- added U1: PIC16F15223, Package_SO:SO-14_3.9x8.65mm_P1.27mm, symbol HandyRadio:PIC16F15223
- renumbered C12 to C10, C14 to C11, C15 to C12, C16 to C14, C17 to C15, C18 to C16, C5 to C2, C6 to C3, C7 to C4, C8 to C6, C9 to C7, C10 to C8, C11 to C9, R11 to R10, R10 to R11, R12 to R13, R13 to R14, R3 to R2, R6 to R3, R5 to R4, R4 to R5, R7 to R6, R8 to R7, R9 to R8, TP5 to TP3, TP6 to TP4, TP3 to TP5, TP7 to TP6, TP8 to TP7, TP9 to TP8, TP4 to TP9
Connections:
- net BEEP_OUPUT is gone; now on net BEEP_SIG: R5.1
- net +3V3: now also R10.2, R14.2, R16.2, U1.1 (VDD); no longer SW1.1, SW2.1, SW3.1
- net BATT_STAT: now also U1.3 (RA4)
- net BEEP_SIG: now also C5.2; no longer R5.2
- net GND: now also R5.2, SW1.2, SW2.2, SW3.2, U1.14 (VSS); no longer R10.1, R14.1
- net I2C_SCL: now also U1.10 (RC0)
- net I2C_SDA: now also U1.9 (RC1)
- net IR_INPUT: now also U1.2 (RA5)
- net LED_IND: now also C5.1, U1.5 (RC5)
- net PB_1: now also R9.2, U1.11 (RA2); no longer C16.2, SW3.2
- net SI47_CLK: now also U1.7 (RC3)
- net ~{FM}/SW_SEL: now also U1.6 (RC4)
- net MCU_NRST renamed ~{MCLR}
- net ~{MCLR}: now also U1.4 (~{MCLR}/VPP/RA3)
- removed net PB_2: C13.2, R14.2, SW2.2
- removed net PB_3: C8.2, R10.2, SW1.2
- net SWCLK renamed ICSPCLK
- net ICSPCLK: now also R12.1, U1.12 (RA1/ICSPCLK)
- net SWDIO: no longer names the net of R3.1
- net SWDIO: now also U1.8 (RC2); no longer J1.3
- new net: C16.2, R15.1, R16.1, SW3.1
- new net: C13.2, R12.2, R14.1, SW2.1
- new net: C8.2, R10.1, R9.1, SW1.1
- new net ICSPDAT: J1.3, R15.2, U1.13 (RA0/ICSPDAT)
- no-connect marks 3 -> 1
Other:
- note removed: "TP List TP1 = MCU_RESET TP2 = GND TP3 = IR_RECEIVER TP4 = BATT_STAT TP5 = I2C_SCL TP6 = I2C_SDA TP7 = GND TP8 = GND TP9 = GND"
- moved on the sheet: C1, C10, C11, C12, C13, C14, C15, C16, C2, C3, C4, C6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

Commit message: layout has been done, only checking rules has been left
Connections:
- net +3.3V is gone; now on net +3V3: D1.2
Changed lines of the file:
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@@
     (pin "2")
+  )
+  (symbol (lib_id "power:+3V3") (at 350.52 212.09 270) (unit 1)
+    (in_bom yes) (on_board yes) (fields_autoplaced)
+    (property "Reference" "#PWR?" (id 0) (at 346.71 212.09 0)
+      (effects (font (size 1.27 1.27)) hide)
+    )
+    (property "Value" "+3V3" (id 1) (at 354.33 212.0899 90)
+      (effects (font (size 1.27 1.27)) (justify left))
+    )
+    (property "Footprint" "" (id 2) (at 350.52 212.09 0)
+      (effects (font (size 1.27 1.27)) hide)
+    )
+    (property "Datasheet" "" (id 3) (at 350.52 212.09 0)
+      (effects (font (size 1.27 1.27)) hide)
+    )
+    (pin "1")
   )
   (symbol (lib_id "power:+3V3") (at 78.74 107.95 90) (unit 1)
@@
       (effects (font (size 1.27 1.27)) hide)
     )
-    (pin "1")
-  )
-  (symbol (lib_id "power:+3.3V") (at 350.52 212.09 270) (unit 1)
-    (in_bom yes) (on_board yes) (fields_autoplaced)
-    (property "Reference" "#PWR021" (id 0) (at 346.71 212.09 0)
-      (effects (font (size 1.27 1.27)) hide)
-    )
-    (property "Value" "+3.3V" (id 1) (at 354.33 212.0899 90)
-      (effects (font (size 1.27 1.27)) (justify left))
-    )
-    (property "Footprint" "" (id 2) (at 350.52 212.09 0)
-      (effects (font (size 1.27 1.27)) hide)
-    )
-    (property "Datasheet" "" (id 3) (at 350.52 212.09 0)
-      (effects (font (size 1.27 1.27)) hide)
-    )

Commit message: some modification
Parts:
- renumbered C1 to C301, C2 to C302, C3 to C303, C4 to C304, C5 to C305, C6 to C306, C7 to C307, C8 to C308, C9 to C309, C10 to C310, C11 to C311, C12 to C312, C13 to C313, C14 to C314, C15 to C315, C16 to C316, D1 to D301, J1 to J301, J2 to J302, R1 to R301, R2 to R302, R3 to R303, R4 to R304, R5 to R305, R6 to R306, R7 to R307, R8 to R308, R9 to R309, R10 to R310, R11 to R311, R12 to R312, R13 to R313, R14 to R314, R15 to R315, R16 to R316, SW1 to SW301, SW2 to SW302, SW3 to SW303, TP1 to TP301, TP2 to TP302, TP3 to TP303, TP4 to TP304, TP5 to TP305, TP6 to TP306, TP7 to TP307, TP8 to TP308, TP9 to TP309, TP10 to TP310, U1 to U301, U2 to U302

Commit message: routing has been almost done
Connections:
- net SI47_CLK: no longer R304.1, U301.7 (RC3)
- new net: R304.1, U301.7 (RC3)
Changed lines of the file:
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@@
-    (effects (font (size 1.27 1.27)) (justify left bottom))
-  )
-  (label "SI47_CLK" (at 167.64 109.22 0)
     (effects (font (size 1.27 1.27)) (justify left bottom))
   )

Commit message: Ready to release the HW :smile:
Other:
- note added: "CHECKED"
- note added: "Design Note: The HPF filter is designed for frequency higher than 160Hz"
- moved on the sheet: C315, R312
