File: HandyRadio/HW/V1_09302022/1- Design Files/_HW_HandyRadio_/[04] - RF RECEIVER.kicad_sch (KiCad schematic)
At the start: 0 parts

Commit message: Schematic is almost done
Parts:
- added ANT?: WHIP_ANT, symbol HandyRadio:WHIP_ANT
- added C? (x3): 33pF, symbol HandyRadio:33pF
- added C? (x2): 6pF, symbol HandyRadio:6pF
- added C? (x2): 3p3F, symbol HandyRadio:3p3F
- added C?: 22nF, symbol HandyRadio:22nF
- added C? (x3): 100nF, symbol HandyRadio:100nF
- added C?: 470nF, symbol HandyRadio:470nF
- added C?: 18pF, symbol HandyRadio:18pF
- added C?: 10nF, symbol HandyRadio:10nF
- added EC? (x2): 4u7F/6.3V, symbol HandyRadio:4u7F{brace}slash}6.3V
- added EC?: 2u2F/10V, symbol HandyRadio:2u2F/10V
- added J?: MHDR_2POS_VERT, symbol HandyRadio:MHDR_2POS_VERT
- added K?: DPDT_RELAY, symbol HandyRadio:DPDT_RELAY
- added L?: 4u7H, symbol HandyRadio:4u7H
- added L? (x2): BLM15GA750SN1D, symbol HandyRadio:BLM15GA750SN1D
- added L?: 180nH, symbol HandyRadio:180nH
- added R? (x3): 10KR, symbol HandyRadio:10KR
- added R? (x2): 330R, symbol HandyRadio:330R
- added R?: 2KR, symbol HandyRadio:2KR
- added R?: 100KR, symbol HandyRadio:100KR
- added U?: SI4735-D60-GU, symbol HandyRadio:SI4735-D60-GU
Connections:
- new net: R?.1, R?.2, U?.15 (~{RST})
- new net: C?.2, R?.1, U?.4 (GPO2/~{INT})
- new net: C?.2, R?.1, U?.5 (GPO1)
- new net: C?.2, L?.2, U?.8 (FMI)
- new net: C?.2, C?.2, L?.1
- new net: C?.2, U?.22 (DBYP)
- new net: C?.1, J?.2, K?.7
- new net: C?.1, C?.2, K?.6
- new net: ANT?.1, C?.1, L?.2
- new net: R?.1, U?.16 (~{SEN})
- new net: C?.2, L?.2, U?.12 (AMI)
- new net: K?.8, L?.1
- new net: C?.2, C?.2, L?.1, L?.1
- new net +3V3: C?.2, EC?.1, R?.2, R?.2, R?.2, R?.2, U?.20 (VIO)
- new net +5V: C?.2, C?.2, EC?.1, EC?.1, U?.21 (VDD)
- new net AUDIO_L: U?.24 (LOUT)
- new net AUDIO_R: U?.23 (ROUT)
- new net FM/SW_SEL: C?.2, K?.4
- new net GND: C?.1, C?.1, C?.1, C?.1, C?.1, C?.1, C?.1, C?.1, C?.1, C?.1, C?.1, EC?.2, EC?.2, EC?.2, J?.1, K?.5, L?.2, R?.1, R?.2, R?.2, U?.13 (GND), U?.14 (GND), U?.9 (RFGND)
- new net I2C_SCL: R?.1, U?.17 (SCLK)
- new net I2C_SDA: R?.1, U?.18 (SDIO)
- no-connect marks 0 -> 8
Other:
- note added: "ADD A BJT"
- note added: "Although the Si4734/35 will respond to only a single device address, this address can be changed with the SEN pin (note that the SEN pin is not used for signaling in 2-wire mode). When SEN = 0, the 7-bit device address is 0010001b. When SEN = 1, the address is 1100011b."
- note added: "DNF"

Commit message: Schematic is almost Done
Parts:
- removed C?: 100nF, symbol HandyRadio:100nF
- added C? (x4): 10uF, symbol HandyRadio:10uF
- added Q?: MMUN2215LT1G, symbol HandyRadio:MMUN2215LT1G
- added TP? (x2): TPC, symbol HandyRadio:TPC
Connections:
- net +3V3: now also K?.4, C?.2, C?.2
- net +5V: now also C?.2, C?.2
- net FM/SW_SEL: now also Q?.1, TP?.1; no longer K?.4
- net GND: now also C?.1, C?.1, C?.1, C?.1, Q?.2, TP?.1; no longer K?.5
- new net: K?.5, Q?.3
Other:
- note added: "INFO:"
- note added: "LAYOUT NOTE:"
- note added: "Q = ON, FM SELECTED Q = OFF, SW SELECTED"
- note added: "The following design checklist summarizes the guidelines presented in this section:  Place bypass caps C1, C2 and C3 as close as possible to the supply and ground pins.  Place a via connecting C1, C2, and C3 to the power supplies such that the cap is between the Si47xx and the via.  Route a wide, low inductance return current path from the C1, C2, and C3 to the Si47xx GND pins.  Route GND/LIN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"
- note added: "The following layout rules are used:  Layer 1 top side placement and routing (shown)  Layer 2 GND (not shown)  Power routed by trace (not shown)  0402 component size or larger  6 mil traces  6 mil trace spacing  15 mil component spacing"
- note added: " Place F1 as close as possible to FMI pin 2.  Place C14 as close as possible to FMI pin 2.  Place C5 even though it is designated as NP, it should be as close as possible to FMI pin2.  On the Si4704/05/06/1x/2x products: Place C4 as close as possible to LPI/TXO pin 4 and RFGND pin 3. Place L1 as close as possible to LPI/TXO pin 4.  On Si473x products: Place C16 as close as possible to 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"
- note removed: "ADD A BJT"
- company: (none) -> Siavash Taher Parvar
- title: (none) -> Handy Radio
- moved on the sheet: ANT?, C?, EC?, J?, K?, L?, R?, U?

Commit message: 95 SCHEMATIC HAS BEEN DONE
Parts:
- added U3: EGUARD0502A, symbol HandyRadio:EGUARD0502A
- gave numbers to parts that had none: 38
Connections:
- net GND: now also U3.2, U3.5
- net at C21.2, K1.6: now also U3.3; no longer C26.1
- net at ANT1.1, L1.2: now also U3.1; no longer C25.1
- new net: C26.1, U3.4
- new net: C25.1, U3.6
Other:
- note added: "Q = OFF, FM SELECTED Q = ON, SW SELECTED"
- note added: " Maximize whip antenna length for optimal performance.  Select matching inductor L1 with a Q of 20 or greater at 25 MHz and minimal dc resistance.  Select L1 inductor value to maximize signal strength across the FM band.  Place L1 and whip antenna close together and as far from potential noise sources as possible to reduce capacitive and inductive coupling.  Place the chip as close as possib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"
- note removed: "Q = ON, FM SELECTED Q = OFF, SW SELECTED"
- moved on the sheet: ANT1, C25, C26, L2

Commit message: Schematic has been double checked
Parts:
- removed L3: BLM15GA750SN1D, symbol HandyRadio:BLM15GA750SN1D
- removed R12, R13: 10KR, symbol HandyRadio:10KR
- added C? (x2): 22nF, symbol HandyRadio:22nF
- added L?: 10nH, symbol HandyRadio:10nH
- added R? (x3): 2KR, symbol HandyRadio:2KR
Connections:
- net +3V3: now also C?.2
- net +5V: now also C?.2
- net GND: now also C?.1, C?.1
- net I2C_SCL: now also R?.1; no longer U4.17 (SCLK)
- net I2C_SDA: now also R?.1; no longer U4.18 (SDIO)
- net ~{RST}: now reaches R14.2, R16.1, U4.15 (~{RST})
- net GPO2: now reaches C34.2, R18.1, U4.4 (GPO2/~{INT})
- net GPO1: now reaches C35.2, R17.1, U4.5 (GPO1)
- net FMI: now reaches C32.2, L4.2, U4.8 (FMI)
- net at C26.2, C28.2: now also L?.1
- net ~{SEN}: now reaches R15.1, U4.16 (~{SEN})
- net AMI: now reaches C31.2, U4.12 (AMI)
- net AMI: now also L?.2
- net RCLK: now reaches U4.19 (RCLK)
- net RCLK: now also R?.2
- new net SCLK: R?.2, U4.17 (SCLK)
- new net SDIO: R?.2, U4.18 (SDIO)
- new net SI47_CLK: R?.1
- no-connect marks 8 -> 10
Other:
- note added: "Place a via connecting C1 VD/VDD supply to the power rail such that the cap is closer to the Si47xx than the via. Route C1 GND directly and only to GND pin 12 with a wide, low inductance trace. C1 GND should not be routed to GND via."
- moved on the sheet: ANT1, C19, C20, C22, C23, C24, C28, C29, C30, C32, EC1, EC2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

Commit message: 99% SCHEMATIC HAS BEEN DONE
Parts:
- gave numbers to parts that had none: 6
- renumbered C22 to C21, C21 to C23, C23 to C24, C24 to C25, C25 to C26, C26 to C27, C29 to C28, C28 to C29, C27 to C30, C30 to C31, C31 to C33, C32 to C34, C33 to C35, C34 to C36, C35 to C37, R14 to R15, R15 to R19, R16 to R20, R17 to R21, R18 to R22, TP10 to TP11, TP11 to TP12

Commit message: almost ready for routing and finishing PCB :D
Parts:
- removed EC1, EC2: 4u7F/6.3V, symbol HandyRadio:4u7F{brace}slash}6.3V
- removed EC3: 2u2F/10V, symbol HandyRadio:2u2F/10V
- added EC? (x2): 4u7F/6.3V, Capacitor_Tantalum_SMD:CP_EIA-2012-12_Kemet-R_Pad1.30x1.05mm_HandSolder, symbol HandyRadio:4u7F/6.3V
- added EC?: 2u2F/10V, Capacitor_Tantalum_SMD:CP_EIA-2012-12_Kemet-R_Pad1.30x1.05mm_HandSolder, symbol HandyRadio:2u2F{brace}slash}10V
- ANT?: renamed from ANT1; footprint (none) -> MountingHole:MountingHole_3.2mm_M3_Pad_Via
- C?: renamed from C25; footprint (none) -> Capacitor_SMD:C_0805_2012Metric_Pad1.18x1.45mm_HandSolder
- C?: renamed from C20; footprint (none) -> Capacitor_SMD:C_0805_2012Metric_Pad1.18x1.45mm_HandSolder
- C?: renamed from C37; footprint (none) -> Capacitor_SMD:C_0805_2012Metric_Pad1.18x1.45mm_HandSolder
- C?: renamed from C34; footprint (none) -> Capacitor_SMD:C_0805_2012Metric_Pad1.18x1.45mm_HandSolder
- C?: renamed from C32; footprint (none) -> Capacitor_SMD:C_0805_2012Metric_Pad1.18x1.45mm_HandSolder
- C?: renamed from C29; footprint (none) -> Capacitor_SMD:C_0805_2012Metric_Pad1.18x1.45mm_HandSolder
- C?: renamed from C22; footprint (none) -> Capacitor_SMD:C_0805_2012Metric_Pad1.18x1.45mm_HandSolder
- C?: renamed from C35; footprint (none) -> Capacitor_SMD:C_0805_2012Metric_Pad1.18x1.45mm_HandSolder
- C?: renamed from C24; footprint (none) -> Capacitor_SMD:C_0805_2012Metric_Pad1.18x1.45mm_HandSolder
- C?: renamed from C21; footprint (none) -> Capacitor_SMD:C_0805_2012Metric_Pad1.18x1.45mm_HandSolder
- C?: renamed from C23; footprint (none) -> Capacitor_SMD:C_0805_2012Metric_Pad1.18x1.45mm_HandSolder
- C?: renamed from C36; footprint (none) -> Capacitor_SMD:C_0805_2012Metric_Pad1.18x1.45mm_HandSolder
- C?: renamed from C27; footprint (none) -> Capacitor_SMD:C_0805_2012Metric_Pad1.18x1.45mm_HandSolder
- C?: renamed from C33; footprint (none) -> Capacitor_SMD:C_0805_2012Metric_Pad1.18x1.45mm_HandSolder
- C?: renamed from C26; footprint (none) -> Capacitor_SMD:C_0805_2012Metric_Pad1.18x1.45mm_HandSolder
- C?: renamed from C30; footprint (none) -> Capacitor_SMD:C_0805_2012Metric_Pad1.18x1.45mm_HandSolder
- C?: renamed from C31; footprint (none) -> Capacitor_SMD:C_0805_2012Metric_Pad1.18x1.45mm_HandSolder
- C?: renamed from C19; footprint (none) -> Capacitor_SMD:C_0805_2012Metric_Pad1.18x1.45mm_HandSolder
- C?: renamed from C28; footprint (none) -> Capacitor_SMD:C_0805_2012Metric_Pad1.18x1.45mm_HandSolder
- J?: renamed from J3; footprint (none) -> Connector_PinHeader_2.54mm:PinHeader_1x02_P2.54mm_Vertical
- K?: renamed from K1; footprint (none) -> Relay_THT:Relay_DPDT_AXICOM_IMSeries_Pitch5.08mm
- L?: renamed from L3; footprint (none) -> Inductor_SMD:L_0603_1608Metric_Pad1.05x0.95mm_HandSolder
- L?: renamed from L1; footprint (none) -> Inductor_SMD:L_0805_2012Metric_Pad1.05x1.20mm_HandSolder
- L?: renamed from L4; footprint (none) -> Inductor_SMD:L_0402_1005Metric_Pad0.77x0.64mm_HandSolder
- L?: renamed from L2; footprint (none) -> Inductor_SMD:L_0603_1608Metric_Pad1.05x0.95mm_HandSolder
- Q?: renamed from Q1; footprint (none) -> Package_TO_SOT_SMD:SOT-23
- R?: renamed from R15; footprint (none) -> Resistor_SMD:R_0805_2012Metric_Pad1.20x1.40mm_HandSolder
- R?: renamed from R22; footprint (none) -> Resistor_SMD:R_0805_2012Metric_Pad1.20x1.40mm_HandSolder
- R?: renamed from R17; footprint (none) -> Resistor_SMD:R_0805_2012Metric_Pad1.20x1.40mm_HandSolder
- R?: renamed from R21; footprint (none) -> Resistor_SMD:R_0805_2012Metric_Pad1.20x1.40mm_HandSolder
- R?: renamed from R16; footprint (none) -> Resistor_SMD:R_0805_2012Metric_Pad1.20x1.40mm_HandSolder
- R?: renamed from R18; footprint (none) -> Resistor_SMD:R_0805_2012Metric_Pad1.20x1.40mm_HandSolder
- R?: renamed from R20; footprint (none) -> Resistor_SMD:R_0805_2012Metric_Pad1.20x1.40mm_HandSolder
- R?: renamed from R19; footprint (none) -> Resistor_SMD:R_0805_2012Metric_Pad1.20x1.40mm_HandSolder
- TP?: renamed from TP12; footprint (none) -> TestPoint:TestPoint_Pad_D1.5mm
- TP?: renamed from TP11; footprint (none) -> TestPoint:TestPoint_Pad_D1.5mm
- U?: renamed from U3; footprint (none) -> Package_TO_SOT_SMD:SOT-563
- U?: renamed from U4; footprint (none) -> Package_SO:SSOP-24_3.9x8.7mm_P0.635mm
Connections:
- net +3V3: now also EC?.1
- net +5V: now also EC?.1, EC?.1
- net GND: now also EC?.2, EC?.2, EC?.2
- net FM/SW_SEL renamed ~{FM}/SW_SEL

Commit message: doing placement
Parts:
- gave numbers to parts that had none: 42
