File: HandyRadio/HW/V1_09302022/1- Design Files/_HW_HandyRadio_/[04] - RF RECEIVER.kicad_sch (KiCad schematic)
At the start: 42 parts, among them J6 MHDR_2POS_VERT, K1 DPDT_RELAY, Q2 MMUN2215LT1G, U8 EGUARD0502A, U9 SI4735-D60-GU

Commit message: serious modification has been done
Parts:
- K1: footprint Relay_THT:Relay_DPDT_AXICOM_IMSeries_Pitch5.08mm -> Relay_THT:Relay_DPDT_Finder_30.22
- renumbered C44 to C52, C45 to C53, C46 to C54, C47 to C55, C48 to C56, C49 to C57, C50 to C58, C51 to C59, C52 to C60, C53 to C61, C54 to C62, C55 to C63, C56 to C64, C57 to C65, C58 to C66, C59 to C67, C60 to C68, C61 to C69, C62 to C70, EC13 to EC4, EC14 to EC5, EC15 to EC6, R33 to R32, R34 to R33, R35 to R34, R36 to R35, R37 to R36, R38 to R37, R39 to R38, R40 to R39
Connections:
- net +3V3: now also K1.A1; no longer K1.4
- net at Q2.3: now also K1.A2; no longer K1.5
- net at C56.2, U8.3: now also K1.21; no longer K1.6
- net at C56.1, J6.2: now also K1.22; no longer K1.7
- net at L2.1: now also K1.24; no longer K1.8

Commit message: some modification
Parts:
- renumbered ANT2 to ANT801, C52 to C801, C53 to C802, C54 to C803, C55 to C804, C56 to C805, C57 to C806, C58 to C807, C59 to C808, C60 to C809, C61 to C810, C62 to C811, C63 to C812, C64 to C813, C65 to C814, C66 to C815, C67 to C816, C68 to C817, C69 to C818, C70 to C819, EC4 to EC801, EC5 to EC802, EC6 to EC803, J6 to J801, K1 to K801, L2 to L801, L3 to L802, L4 to L803, L5 to L804, Q2 to Q801, R32 to R801, R33 to R802, R34 to R803, R35 to R804, R36 to R805, R37 to R806, R38 to R807, R39 to R808, TP20 to TP801, TP21 to TP802, U8 to U801, U9 to U802

Commit message: routing on progress
Parts:
- TC803: renamed from EC803; value 2u2F/10V -> 2u2F/10V; symbol HandyRadio:2u2F{brace}slash}10V -> HandyRadio:2u2F/10V
- renumbered EC801 to TC801, EC802 to TC802
Changed lines of the file:
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@@
   (symbol (lib_id "HandyRadio:4u7F{slash}6.3V") (at 64.77 171.45 270) (unit 1)
     (in_bom yes) (on_board yes) (fields_autoplaced)
-    (property "Reference" "EC801" (id 0) (at 68.58 177.4189 90)
+    (property "Reference" "TC801" (id 0) (at 68.58 177.4189 90)
       (effects (font (size 1.27 1.27)) (justify left))
     )
@@
     (pin "2")
   )
-  (symbol (lib_id "HandyRadio:2u2F{brace}slash}10V") (at 158.75 171.45 270) (unit 1)
-    (in_bom yes) (on_board yes) (fields_autoplaced)
-    (property "Reference" "EC803" (id 0) (at 162.56 177.4189 90)
-      (effects (font (size 1.27 1.27)) (justify left))
-    )
-    (property "Value" "2u2F{slash}10V" (id 1) (at 162.56 179.9589 90)
-      (effects (font (size 1.27 1.27)) (justify left))
-    )
+  (symbol (lib_id "HandyRadio:2u2F{slash}10V") (at 158.75 171.45 270) (unit 1)
+    (in_bom yes) (on_board yes)
+    (property "Reference" "TC803" (id 0) (at 163.83 177.8 90))
+    (property "Value" "2u2F/10V" (id 1) (at 166.37 180.34 90))
     (property "Footprint" "Capacitor_Tantalum_SMD:CP_EIA-2012-12_Kemet-R_Pad1.30x1.05mm_HandSolder" (id 2) (at 166.37 177.8 0)
       (effects (font (size 1.27 1.27)) hide)
@@
   (symbol (lib_id "HandyRadio:4u7F{slash}6.3V") (at 142.24 171.45 270) (unit 1)
     (in_bom yes) (on_board yes) (fields_autoplaced)
-    (property "Reference" "EC802" (id 0) (at 146.05 177.4189 90)
-      (effects (font (size 1.27 1.27)) (justify left))
-    )
+    (property "Reference" "TC802" (id 0) (at 146.05 177.4189 90)
+      (effects (font (size 1.27 1.27)) (justify left))
+    )

Commit message: Ready to release the HW :smile:
Other:
- note added: "CHECKED"
Changed lines of the file:
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@@
   (title_block
     (title "Handy Radio")
+    (date "2022-11-10")
     (rev "01")
     (company "Siavash Taher Parvar")
@@
     (effects (font (size 1.27 1.27)) (justify left bottom))
   )
+  (text "CHECKED" (at 381 36.83 0)
+    (effects (font (size 5 5) (thickness 1) bold) (justify left bottom))
+  )
   (text "LAYOUT NOTE:" (at 154.94 233.68 0)
