File: HandyRadio/HW/V1_09302022/1- Design Files/_HW_HandyRadio_/[05] - AUDIO AMP.kicad_sch (KiCad schematic)
At the start: 0 parts

Commit message: 2/6 HandyRadio HW has been done
Parts:
- added C?: 10nF, symbol HandyRadio:10nF
- added C?: 1uF, symbol HandyRadio:1uF
- added C?: 100nF, symbol HandyRadio:100nF
- added D?: BAT54ATA, symbol HandyRadio:BAT54ATA
- added EC? (x2): 2u2F/10V, symbol HandyRadio:2u2F/10V
- added EC? (x2): 100uF/6.3V, symbol HandyRadio:100uF{brace}slash}6.3V
- added EC?: 4u7F/6.3V, symbol HandyRadio:4u7F{brace}slash}6.3V
- added EC?: 1uF/16V, symbol HandyRadio:1uF/16V
- added J?: AUDIO_Jack, symbol HandyRadio:AUDIO_Jack
- added R? (x2): 100KR, symbol HandyRadio:100KR
- added R? (x2): 1KR, symbol HandyRadio:1KR
- added R? (x4): 3K9R, symbol HandyRadio:3K9R
- added U?: LM4808, symbol HandyRadio:LM4808
Connections:
- new net: EC?.2, J?.3 (RIGHT)
- new net: EC?.2, J?.4 (LEFT)
- new net: EC?.1, R?.1, R?.2, U?.3 (INA+), U?.5 (INB+)
- new net: EC?.1, R?.1 (x2)
- new net: EC?.1, R?.2, U?.7 (OUTB)
- new net: D?.2, R?.1
- new net: EC?.1, R?.2, U?.1 (OUTA)
- new net: R?.1, R?.2, U?.2 (INA-)
- new net: R?.1, R?.2, U?.6 (INB-)
- new net: D?.1, R?.1
- new net +5V: C?.2, C?.2, C?.2, EC?.1, R?.2, U?.8 (VDD)
- new net AUDIO_L: EC?.2, R?.2
- new net AUDIO_R: EC?.2, R?.2
- new net BEEP_SIG: D?.3
- new net GND: C?.1, C?.1, C?.1, EC?.2, EC?.2, J?.2 (GND), R?.1, U?.4 (GND)
- no-connect marks 0 -> 1

Commit message: Schematic is almost Done
Connections:
- net AUDIO_RIGHT: now reaches EC?.2, J?.3 (RIGHT)
- net AUDIO_LEFT: now reaches EC?.2, J?.4 (LEFT)
- net IN+: now reaches EC?.1, R?.1, R?.2, U?.3 (INA+), U?.5 (INB+)
- net INA-: now reaches R?.1, R?.2, U?.2 (INA-)
- net INB-: now reaches R?.1, R?.2, U?.6 (INB-)
Other:
- note added: "LAYOUT:"
- company: (none) -> Siavash Taher Parvar
- title: (none) -> Handy Radio
- moved on the sheet: C?, D?, EC?, J?, R?, U?

Commit message: 95 SCHEMATIC HAS BEEN DONE
Parts:
- gave numbers to parts that had none: 20
Other:
- moved on the sheet: C36, C37, C38, D2, EC4, EC5, EC6, EC7, EC8, EC9, J4, R19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

Commit message: 99% SCHEMATIC HAS BEEN DONE
Parts:
- renumbered C36 to C38, C37 to C39, C38 to C40, R19 to R23, R20 to R24, R21 to R25, R22 to R26, R23 to R27, R24 to R28, R25 to R29, R26 to R30
Changed lines of the file:
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@@
   (symbol (lib_id "HandyRadio:100KR") (at 127 135.89 90) (unit 1)
     (in_bom yes) (on_board yes) (fields_autoplaced)
-    (property "Reference" "R19" (id 0) (at 129.54 126.9999 90)
+    (property "Reference" "R23" (id 0) (at 129.54 126.9999 90)
       (effects (font (size 1.27 1.27)) (justify right))
     )
@@
   (symbol (lib_id "HandyRadio:100KR") (at 127 156.21 90) (unit 1)
     (in_bom yes) (on_board yes) (fields_autoplaced)
-    (property "Reference" "R20" (id 0) (at 129.54 147.3199 90)
+    (property "Reference" "R24" (id 0) (at 129.54 147.3199 90)
       (effects (font (size 1.27 1.27)) (justify right))
     )
@@
   (symbol (lib_id "HandyRadio:10nF") (at 270.51 156.21 90) (unit 1)
     (in_bom yes) (on_board yes) (fields_autoplaced)
-    (property "Reference" "C38" (id 0) (at 274.32 147.3199 90)
+    (property "Reference" "C40" (id 0) (at 274.32 147.3199 90)
       (effects (font (size 1.27 1.27)) (justify right))
     )
@@
   (symbol (lib_id "HandyRadio:1KR") (at 181.61 123.19 0) (unit 1)
     (in_bom yes) (on_board yes)
-    (property "Reference" "R21" (id 0) (at 198.12 121.92 0))
+    (property "Reference" "R25" (id 0) (at 198.12 121.92 0))
     (property "Value" "1KR" (id 1) (at 180.34 121.92 0))
     (property "Footprint" "" (id 2) (at 181.61 123.19 0)
@@
   (symbol (lib_id "HandyRadio:3K9R") (at 303.53 105.41 0) (unit 1)
     (in_bom yes) (on_board yes)
-    (property "Reference" "R25" (id 0) (at 320.04 104.14 0))
+    (property "Reference" "R29" (id 0) (at 320.04 104.14 0))
     (property "Value" "3K9R" (id 1) (at 300.99 104.14 0))
     (property "Footprint" "" (id 2) (at 303.53 105.41 0)
@@
   (symbol (lib_id "HandyRadio:3K9R") (at 267.97 133.35 0) (unit 1)
     (in_bom yes) (on_board yes)
-    (property "Reference" "R24" (id 0) (at 284.48 132.08 0))
+    (property "Reference" "R28" (id 0) (at 284.48 132.08 0))
     (property "Value" "3K9R" (id 1) (at 265.43 132.08 0))
     (property "Footprint" "" (id 2) (at 267.97 133.35 0)
@@
   (symbol (lib_id "HandyRadio:1KR") (at 181.61 128.27 0) (unit 1)
     (in_bom yes) (on_board yes)
-    (property "Reference" "R22" (id 0) (at 198.12 127 0))
+    (property "Reference" "R26" (id 0) (at 198.12 127 0))
     (property "Value" "1KR" (id 1) (at 180.34 127 0))
     (property "Footprint" "" (id 2) (at 181.61 128.27 0)
@@
   (symbol (lib_id "HandyRadio:3K9R") (at 303.53 156.21 0) (unit 1)
     (in_bom yes) (on_board yes)
-    (property "Reference" "R26" (id 0) (at 320.04 154.94 0))
+    (property "Reference" "R30" (id 0) (at 320.04 154.94 0))
     (property "Value" "3K9R" (id 1) (at 300.99 154.94 0))
     (property "Footprint" "" (id 2) (at 303.53 156.21 0)
@@
   (symbol (lib_id "HandyRadio:3K9R") (at 267.97 118.11 0) (unit 1)
     (in_bom yes) (on_board yes)
-    (property "Reference" "R23" (id 0) (at 284.48 116.84 0))
+    (property "Reference" "R27" (id 0) (at 284.48 116.84 0))
     (property "Value" "3K9R" (id 1) (at 265.43 116.84 0))
     (property "Footprint" "" (id 2) (at 267.97 118.11 0)
@@
   (symbol (lib_id "HandyRadio:1uF") (at 241.3 156.21 90) (unit 1)
     (in_bom yes) (on_board yes) (fields_autoplaced)
-    (property "Reference" "C36" (id 0) (at 245.11 147.3199 90)
+    (property "Reference" "C38" (id 0) (at 245.11 147.3199 90)
       (effects (font (size 1.27 1.27)) (justify right))
     )
@@
   (symbol (lib_id "HandyRadio:100nF") (at 255.27 156.21 90) (unit 1)
     (in_bom yes) (on_board yes) (fields_autoplaced)
-    (property "Reference" "C37" (id 0) (at 259.08 147.3199 90)
-      (effects (font (size 1.27 1.27)) (justify right))
-    )
+    (property "Reference" "C39" (id 0) (at 259.08 147.3199 90)
+      (effects (font (size 1.27 1.27)) (justify right))
+    )

Commit message: almost ready for routing and finishing PCB :D
Parts:
- removed EC4: 1uF/16V, symbol HandyRadio:1uF/16V
- removed EC5: 4u7F/6.3V, symbol HandyRadio:4u7F{brace}slash}6.3V
- removed EC6, EC7: 2u2F/10V, symbol HandyRadio:2u2F/10V
- removed EC8, EC9: 100uF/6.3V, symbol HandyRadio:100uF{brace}slash}6.3V
- added EC? (x2): 2u2F/10V, Capacitor_Tantalum_SMD:CP_EIA-2012-12_Kemet-R_Pad1.30x1.05mm_HandSolder, symbol HandyRadio:2u2F{brace}slash}10V
- added EC? (x2): 100uF/6.3V, Capacitor_Tantalum_SMD:CP_EIA-2012-12_Kemet-R_Pad1.30x1.05mm_HandSolder, symbol HandyRadio:100uF/6.3V
- added EC?: 4u7F/6.3V, Capacitor_Tantalum_SMD:CP_EIA-2012-12_Kemet-R_Pad1.30x1.05mm_HandSolder, symbol HandyRadio:4u7F/6.3V
- added EC?: 1uF/16V, Capacitor_Tantalum_SMD:CP_EIA-2012-12_Kemet-R_Pad1.30x1.05mm_HandSolder, symbol HandyRadio:1uF/16V
- C?: renamed from C40; footprint (none) -> Capacitor_SMD:C_0805_2012Metric_Pad1.18x1.45mm_HandSolder
- C?: renamed from C38; footprint (none) -> Capacitor_SMD:C_0805_2012Metric_Pad1.18x1.45mm_HandSolder
- C?: renamed from C39; footprint (none) -> Capacitor_SMD:C_0805_2012Metric_Pad1.18x1.45mm_HandSolder
- D?: renamed from D2; footprint (none) -> Package_TO_SOT_SMD:SOT-23
- J?: renamed from J4; footprint (none) -> Connector_Audio:Jack_3.5mm_CUI_SJ-3523-SMT_Horizontal
- R?: renamed from R23; footprint (none) -> Resistor_SMD:R_0805_2012Metric_Pad1.20x1.40mm_HandSolder
- R?: renamed from R24; footprint (none) -> Resistor_SMD:R_0805_2012Metric_Pad1.20x1.40mm_HandSolder
- R?: renamed from R25; footprint (none) -> Resistor_SMD:R_0805_2012Metric_Pad1.20x1.40mm_HandSolder
- R?: renamed from R29; footprint (none) -> Resistor_SMD:R_0805_2012Metric_Pad1.20x1.40mm_HandSolder
- R?: renamed from R28; footprint (none) -> Resistor_SMD:R_0805_2012Metric_Pad1.20x1.40mm_HandSolder
- R?: renamed from R26; footprint (none) -> Resistor_SMD:R_0805_2012Metric_Pad1.20x1.40mm_HandSolder
- R?: renamed from R30; footprint (none) -> Resistor_SMD:R_0805_2012Metric_Pad1.20x1.40mm_HandSolder
- R?: renamed from R27; footprint (none) -> Resistor_SMD:R_0805_2012Metric_Pad1.20x1.40mm_HandSolder
- U?: renamed from U5; footprint (none) -> Package_SO:SOP-8_3.9x4.9mm_P1.27mm
Connections:
- net +5V: now also EC?.1
- net AUDIO_L: now also EC?.2
- net AUDIO_LEFT: now also J?.T (LEFT), EC?.2; no longer J?.4 (LEFT)
- net AUDIO_R: now also EC?.2
- net AUDIO_RIGHT: now also J?.R (RIGHT), EC?.2; no longer J?.3 (RIGHT)
- net GND: now also J?.S (GND), EC?.2, EC?.2; no longer J?.2 (GND)
- net IN+: now also EC?.1
- net at R?.1: now also EC?.1 (x2)
- net at R?.2, U?.7 (OUTB): now also EC?.1
- net at R?.2, U?.1 (OUTA): now also EC?.1
- no-connect marks 1 -> 0

Commit message: doing placement
Parts:
- gave numbers to parts that had none: 20
Changed lines of the file:
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@@
   (symbol (lib_id "HandyRadio:AUDIO_Jack") (at 391.16 121.92 0) (unit 1)
     (in_bom yes) (on_board yes) (fields_autoplaced)
-    (property "Reference" "J?" (id 0) (at 403.86 126.9999 0)
+    (property "Reference" "J3" (id 0) (at 403.86 126.9999 0)
       (effects (font (size 1.27 1.27)) (justify left))
     )
@@
   (symbol (lib_id "HandyRadio:2u2F{brace}slash}10V") (at 250.19 118.11 180) (unit 1)
     (in_bom yes) (on_board yes)
-    (property "Reference" "EC?" (id 0) (at 251.46 116.84 0))
+    (property "Reference" "EC3" (id 0) (at 251.46 116.84 0))
     (property "Value" "2u2F{slash}10V" (id 1) (at 231.14 116.84 0))
     (property "Footprint" "Capacitor_Tantalum_SMD:CP_EIA-2012-12_Kemet-R_Pad1.30x1.05mm_HandSolder" (id 2) (at 243.84 125.73 0)
@@
   (symbol (lib_id "HandyRadio:100KR") (at 127 135.89 90) (unit 1)
     (in_bom yes) (on_board yes) (fields_autoplaced)
-    (property "Reference" "R?" (id 0) (at 129.54 126.9999 90)
+    (property "Reference" "R15" (id 0) (at 129.54 126.9999 90)
       (effects (font (size 1.27 1.27)) (justify right))
     )
@@
   (symbol (lib_id "power:GND") (at 372.11 134.62 0) (unit 1)
     (in_bom yes) (on_board yes) (fields_autoplaced)
-    (property "Reference" "#PWR?" (id 0) (at 372.11 140.97 0)
+    (property "Reference" "#PWR030" (id 0) (at 372.11 140.97 0)
       (effects (font (size 1.27 1.27)) hide)
     )
@@
   (symbol (lib_id "power:+5V") (at 127 118.11 0) (unit 1)
     (in_bom yes) (on_board yes) (fields_autoplaced)
-    (property "Reference" "#PWR?" (id 0) (at 127 121.92 0)
+    (property "Reference" "#PWR026" (id 0) (at 127 121.92 0)
       (effects (font (size 1.27 1.27)) hide)
     )
@@
   (symbol (lib_id "HandyRadio:100KR") (at 127 156.21 90) (unit 1)
     (in_bom yes) (on_board yes) (fields_autoplaced)
-    (property "Reference" "R?" (id 0) (at 129.54 147.3199 90)
+    (property "Reference" "R16" (id 0) (at 129.54 147.3199 90)
       (effects (font (size 1.27 1.27)) (justify right))
     )
@@
   (symbol (lib_id "HandyRadio:2u2F{brace}slash}10V") (at 250.19 133.35 180) (unit 1)
     (in_bom yes) (on_board yes)
-    (property "Reference" "EC?" (id 0) (at 251.46 132.08 0))
+    (property "Reference" "EC4" (id 0) (at 251.46 132.08 0))
     (property "Value" "2u2F{slash}10V" (id 1) (at 231.14 132.08 0))
     (property "Footprint" "Capacitor_Tantalum_SMD:CP_EIA-2012-12_Kemet-R_Pad1.30x1.05mm_HandSolder" (id 2) (at 243.84 140.97 0)
@@
   (symbol (lib_id "HandyRadio:100uF{slash}6.3V") (at 342.9 130.81 0) (unit 1)
     (in_bom yes) (on_board yes)
-    (property "Reference" "EC?" (id 0) (at 359.41 129.54 0))
+    (property "Reference" "EC6" (id 0) (at 359.41 129.54 0))
     (property "Value" "100uF/6.3V" (id 1) (at 337.82 129.54 0))
     (property "Footprint" "Capacitor_Tantalum_SMD:CP_EIA-2012-12_Kemet-R_Pad1.30x1.05mm_HandSolder" (id 2) (at 347.98 125.73 0)
@@
   (symbol (lib_id "power:+5V") (at 217.17 138.43 90) (unit 1)
     (in_bom yes) (on_board yes) (fields_autoplaced)
-    (property "Reference" "#PWR?" (id 0) (at 220.98 138.43 0)
+    (property "Reference" "#PWR028" (id 0) (at 220.98 138.43 0)
       (effects (font (size 1.27 1.27)) hide)
     )
@@
   (symbol (lib_id "HandyRadio:10nF") (at 270.51 156.21 90) (unit 1)
     (in_bom yes) (on_board yes) (fields_autoplaced)
-    (property "Reference" "C?" (id 0) (at 274.32 147.3199 90)
+    (property "Reference" "C21" (id 0) (at 274.32 147.3199 90)
       (effects (font (size 1.27 1.27)) (justify right))
     )
@@
   (symbol (lib_id "HandyRadio:1KR") (at 181.61 123.19 0) (unit 1)
     (in_bom yes) (on_board yes)
-    (property "Reference" "R?" (id 0) (at 198.12 121.92 0))
+    (property "Reference" "R17" (id 0) (at 198.12 121.92 0))
     (property "Value" "1KR" (id 1) (at 180.34 121.92 0))
     (property "Footprint" "Resistor_SMD:R_0805_2012Metric_Pad1.20x1.40mm_HandSolder" (id 2) (at 181.61 123.19 0)
@@
   (symbol (lib_id "HandyRadio:3K9R") (at 303.53 105.41 0) (unit 1)
     (in_bom yes) (on_board yes)
-    (property "Reference" "R?" (id 0) (at 320.04 104.14 0))
+    (property "Reference" "R21" (id 0) (at 320.04 104.14 0))
     (property "Value" "3K9R" (id 1) (at 300.99 104.14 0))
     (property "Footprint" "Resistor_SMD:R_0805_2012Metric_Pad1.20x1.40mm_HandSolder" (id 2) (at 303.53 105.41 0)
@@
   (symbol (lib_id "HandyRadio:LM4808") (at 306.07 115.57 0) (unit 1)
     (in_bom yes) (on_board yes) (fields_autoplaced)
-    (property "Reference" "U?" (id 0) (at 312.42 110.49 0))
+    (property "Reference" "U3" (id 0) (at 312.42 110.49 0))
     (property "Value" "LM4808" (id 1) (at 312.42 113.03 0))
     (property "Footprint" "Package_SO:SOP-8_3.9x4.9mm_P1.27mm" (id 2) (at 306.07 115.57 0)
@@
   (symbol (lib_id "power:GND") (at 222.25 160.02 0) (unit 1)
     (in_bom yes) (on_board yes) (fields_autoplaced)
-    (property "Reference" "#PWR?" (id 0) (at 222.25 166.37 0)
+    (property "Reference" "#PWR029" (id 0) (at 222.25 166.37 0)
       (effects (font (size 1.27 1.27)) hide)
     )
@@
   (symbol (lib_id "HandyRadio:3K9R") (at 267.97 133.35 0) (unit 1)
     (in_bom yes) (on_board yes)
-    (property "Reference" "R?" (id 0) (at 284.48 132.08 0))
+    (property "Reference" "R20" (id 0) (at 284.48 132.08 0))
     (property "Value" "3K9R" (id 1) (at 265.43 132.08 0))
     (property "Footprint" "Resistor_SMD:R_0805_2012Metric_Pad1.20x1.40mm_HandSolder" (id 2) (at 267.97 133.35 0)
@@
   (symbol (lib_id "HandyRadio:4u7F{slash}6.3V") (at 222.25 140.97 270) (unit 1)
     (in_bom yes) (on_board yes) (fields_autoplaced)
-    (property "Reference" "EC?" (id 0) (at 226.06 146.9389 90)
+    (property "Reference" "EC2" (id 0) (at 226.06 146.9389 90)
       (effects (font (size 1.27 1.27)) (justify left))
     )
@@
   (symbol (lib_id "HandyRadio:1KR") (at 181.61 128.27 0) (unit 1)
     (in_bom yes) (on_board yes)
-    (property "Reference" "R?" (id 0) (at 198.12 127 0))
+    (property "Reference" "R18" (id 0) (at 198.12 127 0))
     (property "Value" "1KR" (id 1) (at 180.34 127 0))
     (property "Footprint" "Resistor_SMD:R_0805_2012Metric_Pad1.20x1.40mm_HandSolder" (id 2) (at 181.61 128.27 0)
@@
   (symbol (lib_id "HandyRadio:3K9R") (at 303.53 156.21 0) (unit 1)
     (in_bom yes) (on_board yes)
-    (property "Reference" "R?" (id 0) (at 320.04 154.94 0))
+    (property "Reference" "R22" (id 0) (at 320.04 154.94 0))
     (property "Value" "3K9R" (id 1) (at 300.99 154.94 0))
     (property "Footprint" "Resistor_SMD:R_0805_2012Metric_Pad1.20x1.40mm_HandSolder" (id 2) (at 303.53 156.21 0)
@@
   (symbol (lib_id "HandyRadio:3K9R") (at 267.97 118.11 0) (unit 1)
     (in_bom yes) (on_board yes)
-    (property "Reference" "R?" (id 0) (at 284.48 116.84 0))
+    (property "Reference" "R19" (id 0) (at 284.48 116.84 0))
     (property "Value" "3K9R" (id 1) (at 265.43 116.84 0))
     (property "Footprint" "Resistor_SMD:R_0805_2012Metric_Pad1.20x1.40mm_HandSolder" (id 2) (at 267.97 118.11 0)
@@
   (symbol (lib_id "HandyRadio:100uF{slash}6.3V") (at 342.9 120.65 0) (unit 1)
     (in_bom yes) (on_board yes)
-    (property "Reference" "EC?" (id 0) (at 359.41 119.38 0))
+    (property "Reference" "EC5" (id 0) (at 359.41 119.38 0))
     (property "Value" "100uF/6.3V" (id 1) (at 337.82 119.38 0))
     (property "Footprint" "Capacitor_Tantalum_SMD:CP_EIA-2012-12_Kemet-R_Pad1.30x1.05mm_HandSolder" (id 2) (at 347.98 115.57 0)
@@
   (symbol (lib_id "HandyRadio:1uF") (at 241.3 156.21 90) (unit 1)
     (in_bom yes) (on_board yes) (fields_autoplaced)
-    (property "Reference" "C?" (id 0) (at 245.11 147.3199 90)
+    (property "Reference" "C19" (id 0) (at 245.11 147.3199 90)
       (effects (font (size 1.27 1.27)) (justify right))
     )
@@
   (symbol (lib_id "power:GND") (at 127 160.02 0) (unit 1)
     (in_bom yes) (on_board yes) (fields_autoplaced)
-    (property "Reference" "#PWR?" (id 0) (at 127 166.37 0)
+    (property "Reference" "#PWR027" (id 0) (at 127 166.37 0)
       (effects (font (size 1.27 1.27)) hide)
     )
@@
   (symbol (lib_id "HandyRadio:1uF{slash}16V") (at 142.24 140.97 270) (unit 1)
     (in_bom yes) (on_board yes) (fields_autoplaced)
-    (property "Reference" "EC?" (id 0) (at 146.05 146.9389 90)
+    (property "Reference" "EC1" (id 0) (at 146.05 146.9389 90)
       (effects (font (size 1.27 1.27)) (justify left))
     )
@@
   (symbol (lib_id "HandyRadio:100nF") (at 255.27 156.21 90) (unit 1)
     (in_bom yes) (on_board yes) (fields_autoplaced)
-    (property "Reference" "C?" (id 0) (at 259.08 147.3199 90)
+    (property "Reference" "C20" (id 0) (at 259.08 147.3199 90)
       (effects (font (size 1.27 1.27)) (justify right))
     )
@@
   (symbol (lib_id "HandyRadio:BAT54ATA") (at 161.29 123.19 0) (unit 1)
     (in_bom yes) (on_board yes)
-    (property "Reference" "D?" (id 0) (at 170.18 115.57 0))
+    (property "Reference" "D2" (id 0) (at 170.18 115.57 0))
     (property "Value" "BAT54ATA" (id 1) (at 170.18 118.11 0))
     (property "Footprint" "Package_TO_SOT_SMD:SOT-23" (id 2) (at 161.29 123.19 0)

Commit message: Working on lib and pcb layout
Parts:
- J3: footprint Connector_Audio:Jack_3.5mm_CUI_SJ-3523-SMT_Horizontal -> _HW_HandyRadio_Footprint:Jack_3.5mm_CUI_SJ-3524-SMT_Horizontal
- U3: footprint Package_SO:SOP-8_3.9x4.9mm_P1.27mm -> _HW_HandyRadio_Footprint:SOP-8_3.9x4.9mm_P1.27mm
Changed lines of the file:
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@@
       (effects (font (size 1.27 1.27)) (justify left))
     )
-    (property "Footprint" "Connector_Audio:Jack_3.5mm_CUI_SJ-3523-SMT_Horizontal" (id 2) (at 391.16 121.92 0)
+    (property "Footprint" "_HW_HandyRadio_Footprint:Jack_3.5mm_CUI_SJ-3524-SMT_Horizontal" (id 2) (at 391.16 121.92 0)
       (effects (font (size 1.27 1.27)) hide)
     )
@@
     (property "Reference" "U3" (id 0) (at 312.42 110.49 0))
     (property "Value" "LM4808" (id 1) (at 312.42 113.03 0))
-    (property "Footprint" "Package_SO:SOP-8_3.9x4.9mm_P1.27mm" (id 2) (at 306.07 115.57 0)
-      (effects (font (size 1.27 1.27)) hide)
-    )
+    (property "Footprint" "_HW_HandyRadio_Footprint:SOP-8_3.9x4.9mm_P1.27mm" (id 2) (at 306.07 115.57 0)
+      (effects (font (size 1.27 1.27)) hide)
+    )
