File: HandyRadio/HW/V1_09302022/1- Design Files/_HW_HandyRadio_/[05] - AUDIO AMP.kicad_sch (KiCad schematic)
At the start: 20 parts, among them J3 AUDIO_Jack, U3 LM4808

Commit message: serious modification has been done
Parts:
- removed D2: BAT54ATA, Package_TO_SOT_SMD:SOT-23, symbol HandyRadio:BAT54ATA
- removed EC1: 1uF/16V, Capacitor_Tantalum_SMD:CP_EIA-2012-12_Kemet-R_Pad1.30x1.05mm_HandSolder, symbol HandyRadio:1uF/16V
- removed EC2: 4u7F/6.3V, Capacitor_Tantalum_SMD:CP_EIA-2012-12_Kemet-R_Pad1.30x1.05mm_HandSolder, symbol HandyRadio:4u7F/6.3V
- removed EC3, EC4: 2u2F/10V, Capacitor_Tantalum_SMD:CP_EIA-2012-12_Kemet-R_Pad1.30x1.05mm_HandSolder, symbol HandyRadio:2u2F{brace}slash}10V
- removed EC5, EC6: 100uF/6.3V, Capacitor_Tantalum_SMD:CP_EIA-2012-12_Kemet-R_Pad1.30x1.05mm_HandSolder, symbol HandyRadio:100uF/6.3V
- removed J3: AUDIO_Jack, _HW_HandyRadio_Footprint:Jack_3.5mm_CUI_SJ-3524-SMT_Horizontal, symbol HandyRadio:AUDIO_Jack
- removed R15, R16: 100KR, Resistor_SMD:R_0805_2012Metric_Pad1.20x1.40mm_HandSolder, symbol HandyRadio:100KR
- removed R17, R18: 1KR, Resistor_SMD:R_0805_2012Metric_Pad1.20x1.40mm_HandSolder, symbol HandyRadio:1KR
- removed R21, R22: 3K9R, Resistor_SMD:R_0805_2012Metric_Pad1.20x1.40mm_HandSolder, symbol HandyRadio:3K9R
- removed U3: LM4808, _HW_HandyRadio_Footprint:SOP-8_3.9x4.9mm_P1.27mm, symbol HandyRadio:LM4808
- added C17: 10uF, Capacitor_SMD:C_0805_2012Metric_Pad1.18x1.45mm_HandSolder, symbol HandyRadio:10uF
- added C20, C21, C22: 100nF, Capacitor_SMD:C_0805_2012Metric_Pad1.18x1.45mm_HandSolder, symbol HandyRadio:100nF
- added J3: XH_CONN_2POS_R/A, Connector_JST:JST_PH_S2B-PH-K_1x02_P2.00mm_Horizontal, symbol HandyRadio:XH_CONN_2POS_R/A
- added R19: 10KR, Resistor_SMD:R_0805_2012Metric_Pad1.20x1.40mm_HandSolder, symbol HandyRadio:10KR
- added U3: PAM8302AASCR, Package_SO:MSOP-8_3x3mm_P0.65mm, symbol HandyRadio:PAM8302AASCR
- renumbered C19 to C18, C20 to C19, C21 to C23, R19 to R17, R20 to R18
Connections:
- net INB- is gone; now on an unnamed net: R18.2
- net +5V: now also C17.1, R19.1, U3.6 (VDD)
- net AUDIO_L: now also R17.1
- net AUDIO_R: now also R18.1
- net BEEP_SIG: now also C20.1
- net GND: now also C17.2, C22.1, U3.7 (GND)
- net INA-: no longer names the net of R17.2
- net INA-: now also C21.1
- new net: R19.2, U3.1 (~{SD})
- new net: C20.2, C21.2, U3.3 (IN+)
- new net: C22.2, U3.4 (IN-)
- new net SPK+: J3.1, U3.5 (VO+)
- new net SPK-: J3.2, U3.8 (VO-)
- no-connect marks 0 -> 1
Other:
- note removed: "LAYOUT:"
- moved on the sheet: C18, C19, C23, R17, R18

Commit message: some modification
Parts:
- renumbered C17 to C401, C18 to C402, C19 to C403, C20 to C404, C21 to C405, C22 to C406, C23 to C407, J3 to J401, R17 to R401, R18 to R402, R19 to R403, U3 to U401
Changed lines of the file:
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@@
   (symbol (lib_id "HandyRadio:XH_CONN_2POS_R{slash}A") (at 264.16 110.49 0) (unit 1)
     (in_bom yes) (on_board yes) (fields_autoplaced)
-    (property "Reference" "J3" (id 0) (at 270.51 113.0299 0)
+    (property "Reference" "J401" (id 0) (at 270.51 113.0299 0)
       (effects (font (size 1.27 1.27)) (justify left))
     )
@@
   (symbol (lib_id "HandyRadio:PAM8302AASCR") (at 233.68 110.49 0) (unit 1)
     (in_bom yes) (on_board yes) (fields_autoplaced)
-    (property "Reference" "U3" (id 0) (at 240.03 105.41 0))
+    (property "Reference" "U401" (id 0) (at 240.03 105.41 0))
     (property "Value" "PAM8302AASCR" (id 1) (at 240.03 107.95 0))
     (property "Footprint" "Package_SO:MSOP-8_3x3mm_P0.65mm" (id 2) (at 241.3 104.14 0)
@@
   (symbol (lib_id "HandyRadio:100nF") (at 191.77 110.49 0) (unit 1)
     (in_bom yes) (on_board yes)
-    (property "Reference" "C21" (id 0) (at 208.28 109.22 0))
+    (property "Reference" "C405" (id 0) (at 208.28 109.22 0))
     (property "Value" "100nF" (id 1) (at 189.23 109.22 0))
     (property "Footprint" "Capacitor_SMD:C_0805_2012Metric_Pad1.18x1.45mm_HandSolder" (id 2) (at 203.2 99.06 0)
@@
   (symbol (lib_id "power:+5V") (at 144.78 120.65 90) (unit 1)
     (in_bom yes) (on_board yes) (fields_autoplaced)
-    (property "Reference" "#PWR024" (id 0) (at 148.59 120.65 0)
+    (property "Reference" "#PWR0401" (id 0) (at 148.59 120.65 0)
       (effects (font (size 1.27 1.27)) hide)
     )
@@
   (symbol (lib_id "HandyRadio:10nF") (at 198.12 138.43 90) (unit 1)
     (in_bom yes) (on_board yes) (fields_autoplaced)
-    (property "Reference" "C23" (id 0) (at 201.93 129.5399 90)
+    (property "Reference" "C407" (id 0) (at 201.93 129.5399 90)
       (effects (font (size 1.27 1.27)) (justify right))
     )
@@
   (symbol (lib_id "HandyRadio:10KR") (at 191.77 118.11 0) (unit 1)
     (in_bom yes) (on_board yes)
-    (property "Reference" "R19" (id 0) (at 208.28 116.84 0))
+    (property "Reference" "R403" (id 0) (at 208.28 116.84 0))
     (property "Value" "10KR" (id 1) (at 189.23 116.84 0))
     (property "Footprint" "Resistor_SMD:R_0805_2012Metric_Pad1.20x1.40mm_HandSolder" (id 2) (at 191.77 118.11 0)
@@
   (symbol (lib_id "power:GND") (at 149.86 113.03 270) (unit 1)
     (in_bom yes) (on_board yes) (fields_autoplaced)
-    (property "Reference" "#PWR025" (id 0) (at 143.51 113.03 0)
+    (property "Reference" "#PWR0402" (id 0) (at 143.51 113.03 0)
       (effects (font (size 1.27 1.27)) hide)
     )
@@
   (symbol (lib_id "power:GND") (at 149.86 142.24 0) (unit 1)
     (in_bom yes) (on_board yes) (fields_autoplaced)
-    (property "Reference" "#PWR026" (id 0) (at 149.86 148.59 0)
+    (property "Reference" "#PWR0403" (id 0) (at 149.86 148.59 0)
       (effects (font (size 1.27 1.27)) hide)
     )
@@
   (symbol (lib_id "HandyRadio:3K9R") (at 160.02 110.49 0) (unit 1)
     (in_bom yes) (on_board yes)
-    (property "Reference" "R18" (id 0) (at 176.53 109.22 0))
+    (property "Reference" "R402" (id 0) (at 176.53 109.22 0))
     (property "Value" "3K9R" (id 1) (at 157.48 109.22 0))
     (property "Footprint" "Resistor_SMD:R_0805_2012Metric_Pad1.20x1.40mm_HandSolder" (id 2) (at 160.02 110.49 0)
@@
   (symbol (lib_id "HandyRadio:100nF") (at 191.77 105.41 0) (unit 1)
     (in_bom yes) (on_board yes)
-    (property "Reference" "C20" (id 0) (at 208.28 104.14 0))
+    (property "Reference" "C404" (id 0) (at 208.28 104.14 0))
     (property "Value" "100nF" (id 1) (at 189.23 104.14 0))
     (property "Footprint" "Capacitor_SMD:C_0805_2012Metric_Pad1.18x1.45mm_HandSolder" (id 2) (at 203.2 93.98 0)
@@
   (symbol (lib_id "HandyRadio:3K9R") (at 160.02 107.95 0) (unit 1)
     (in_bom yes) (on_board yes)
-    (property "Reference" "R17" (id 0) (at 176.53 106.68 0))
+    (property "Reference" "R401" (id 0) (at 176.53 106.68 0))
     (property "Value" "3K9R" (id 1) (at 157.48 106.68 0))
     (property "Footprint" "Resistor_SMD:R_0805_2012Metric_Pad1.20x1.40mm_HandSolder" (id 2) (at 160.02 107.95 0)
@@
   (symbol (lib_id "HandyRadio:100nF") (at 191.77 113.03 0) (unit 1)
     (in_bom yes) (on_board yes)
-    (property "Reference" "C22" (id 0) (at 208.28 111.76 0))
+    (property "Reference" "C406" (id 0) (at 208.28 111.76 0))
     (property "Value" "100nF" (id 1) (at 189.23 111.76 0))
     (property "Footprint" "Capacitor_SMD:C_0805_2012Metric_Pad1.18x1.45mm_HandSolder" (id 2) (at 203.2 101.6 0)
@@
   (symbol (lib_id "HandyRadio:1uF") (at 168.91 138.43 90) (unit 1)
     (in_bom yes) (on_board yes) (fields_autoplaced)
-    (property "Reference" "C18" (id 0) (at 172.72 129.5399 90)
+    (property "Reference" "C402" (id 0) (at 172.72 129.5399 90)
       (effects (font (size 1.27 1.27)) (justify right))
     )
@@
   (symbol (lib_id "HandyRadio:10uF") (at 149.86 123.19 270) (unit 1)
     (in_bom yes) (on_board yes) (fields_autoplaced)
-    (property "Reference" "C17" (id 0) (at 153.67 129.5399 90)
+    (property "Reference" "C401" (id 0) (at 153.67 129.5399 90)
       (effects (font (size 1.27 1.27)) (justify left))
     )
@@
   (symbol (lib_id "HandyRadio:100nF") (at 182.88 138.43 90) (unit 1)
     (in_bom yes) (on_board yes) (fields_autoplaced)
-    (property "Reference" "C19" (id 0) (at 186.69 129.5399 90)
-      (effects (font (size 1.27 1.27)) (justify right))
-    )
+    (property "Reference" "C403" (id 0) (at 186.69 129.5399 90)
+      (effects (font (size 1.27 1.27)) (justify right))
+    )

Commit message: Ready to release the HW :smile:
Other:
- note added: "CHECKED"
Changed lines of the file:
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@@
   (title_block
     (title "Handy Radio")
+    (date "2022-11-10")
     (rev "01")
     (company "Siavash Taher Parvar")
@@
     (stroke (width 0) (type default) (color 0 0 0 0))
   )
+  (text "CHECKED" (at 375.92 38.1 0)
+    (effects (font (size 5 5) (thickness 1) bold) (justify left bottom))
+  )
   (label "SPK-" (at 252.73 115.57 0)
