File: HandyRadio/HW/V1_09302022/1- Design Files/_HW_HandyRadio_/_HW_HandyRadio_.kicad_sch (KiCad schematic)
At the start: 0 parts

Commit message: almost ready for routing and finishing PCB :D
Other:
- removed sheet AUDIO AMP
- removed sheet DCDC PWS
- removed sheet MCU, RTC, OLED, PB, LED
- removed sheet RF RECEIVER
- note added: "AUDIO AMP"
- note added: "DCDC PWS"
- note added: "MCU, RTC, OLED, PB, LED"
- note added: "RF RECEIVER"
