File: HandyRadio/HW/V1_09302022/1- Design Files/_HW_HandyRadio_/_HW_HandyRadio_.kicad_sch (KiCad schematic)
At the start: 0 parts

Commit message: Ready to release the HW :smile:
Changed lines of the file:
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@@
   (title_block
     (title "Handy Radio")
+    (date "2022-11-10")
     (rev "01")
     (company "Siavash Taher Parvar")
