File: HandyRadio/HW/V1_09302022/1- Design Files/_HW_HandyRadio_/[07] - MECHANICAL PARTS.kicad_sch (KiCad schematic)
At the start: 0 parts

Commit message: 99% SCHEMATIC HAS BEEN DONE
Parts:
- added ANT2: FERRITE_ANTENNA, symbol HandyRadio:FERRITE_ANTENNA
- added BATT1: Li-PO_BATTERY, symbol HandyRadio:Li-PO_BATTERY
- added DIS1: OLED, symbol HandyRadio:OLED
- added H1: BOX, symbol HandyRadio:BOX
- added H2, H3, H4, H5: SCREW_HOLE, symbol HandyRadio:SCREW_HOLE
- added LBL1: LABLES, symbol HandyRadio:LABLES
- added LS1: HEADPHONE, symbol HandyRadio:HEADPHONE
- added PCB1: PCB, symbol HandyRadio:PCB
Other:
- note removed: "add an OLED display add a Ferrite bead antenna add a earpod add a lithium battery add a box add a PCB add labels"
Changed lines of the file:
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@@
     (comment 9 "N/A")
   )
-  (text "add an OLED display\n\nadd a Ferrite bead antenna\n\nadd a earpod\n\nadd a lithium battery\n\nadd a box\n\nadd a PCB\n\nadd labels"
-    (at 134.62 163.83 0)
-    (effects (font (size 3 3)) (justify left bottom))
+  (symbol (lib_id "HandyRadio:LABLES") (at 195.58 76.2 0) (unit 1)
+    (in_bom no) (on_board no) (fields_autoplaced)
+    (property "Reference" "LBL1" (id 0) (at 238.76 82.5499 0)
+      (effects (font (size 1.27 1.27)) (justify left))
+    )
+    (property "Value" "LABLES" (id 1) (at 238.76 85.0899 0)
+      (effects (font (size 1.27 1.27)) (justify left))
+    )
+    (property "Footprint" "" (id 2) (at 200.66 71.12 0)
+      (effects (font (size 1.27 1.27)) hide)
+    )
+    (property "Datasheet" "" (id 3) (at 200.66 71.12 0)
+      (effects (font (size 1.27 1.27)) hide)
+    )
+  )
+  (symbol (lib_id "HandyRadio:Li-PO_BATTERY") (at 104.14 194.31 0) (unit 1)
+    (in_bom yes) (on_board yes) (fields_autoplaced)
+    (property "Reference" "BATT1" (id 0) (at 122.555 189.23 0))
+    (property "Value" "Li-PO_BATTERY" (id 1) (at 122.555 191.77 0))
+    (property "Footprint" "" (id 2) (at 109.22 185.42 0)
+      (effects (font (size 1.27 1.27)) hide)
+    )
+    (property "Datasheet" "https://www.amazon.ca/Fytoo-300mah-Li-Battery-Control-Battery/dp/B08MW2YGS2/ref=sr_1_1_sspa?keywords=3+7v+300mah&qid=1665512743&qu=eyJxc2MiOiIyLjU3IiwicXNhIjoiMi4zMSIsInFzcCI6IjIuMzIifQ%3D%3D&sprefix=3.7v%2Caps%2C87&sr=8-1-spons&psc=1&smid=AQ7920MIUJ04Q" (id 3) (at 109.22 185.42 0)
+      (effects (font (size 1.27 1.27)) hide)
+    )
+    (property "Description" "Li-PO battery, 3.7V, 300mA" (id 4) (at 109.22 185.42 0)
+      (effects (font (size 1.27 1.27)) hide)
+    )
+  )
+  (symbol (lib_id "HandyRadio:SCREW_HOLE") (at 287.02 78.74 0) (unit 1)
+    (in_bom no) (on_board yes) (fields_autoplaced)
+    (property "Reference" "H2" (id 0) (at 292.1 77.4699 0)
+      (effects (font (size 1.27 1.27)) (justify left))
+    )
+    (property "Value" "SCREW_HOLE" (id 1) (at 292.1 80.0099 0)
+      (effects (font (size 1.27 1.27)) (justify left))
+    )
+    (property "Footprint" "" (id 2) (at 294.64 73.66 0)
+      (effects (font (size 1.27 1.27)) hide)
+    )
+    (property "Datasheet" "" (id 3) (at 294.64 73.66 0)
+      (effects (font (size 1.27 1.27)) hide)
+    )
+    (property "Description" "3.5MM SCREW HOLE_WITHOUT NET" (id 4) (at 294.64 73.66 0)
+      (effects (font (size 1.27 1.27)) hide)
+    )
+  )
+  (symbol (lib_id "HandyRadio:SCREW_HOLE") (at 311.15 78.74 0) (unit 1)
+    (in_bom no) (on_board yes) (fields_autoplaced)
+    (property "Reference" "H4" (id 0) (at 316.23 77.4699 0)
+      (effects (font (size 1.27 1.27)) (justify left))
+    )
+    (property "Value" "SCREW_HOLE" (id 1) (at 316.23 80.0099 0)
+      (effects (font (size 1.27 1.27)) (justify left))
+    )
+    (property "Footprint" "" (id 2) (at 318.77 73.66 0)
+      (effects (font (size 1.27 1.27)) hide)
+    )
+    (property "Datasheet" "" (id 3) (at 318.77 73.66 0)
+      (effects (font (size 1.27 1.27)) hide)
+    )
+    (property "Description" "3.5MM SCREW HOLE_WITHOUT NET" (id 4) (at 318.77 73.66 0)
+      (effects (font (size 1.27 1.27)) hide)
+    )
+  )
+  (symbol (lib_id "HandyRadio:SCREW_HOLE") (at 311.15 90.17 0) (unit 1)
+    (in_bom no) (on_board yes) (fields_autoplaced)
+    (property "Reference" "H5" (id 0) (at 316.23 88.8999 0)
+      (effects (font (size 1.27 1.27)) (justify left))
+    )
+    (property "Value" "SCREW_HOLE" (id 1) (at 316.23 91.4399 0)
+      (effects (font (size 1.27 1.27)) (justify left))
+    )
+    (property "Footprint" "" (id 2) (at 318.77 85.09 0)
+      (effects (font (size 1.27 1.27)) hide)
+    )
+    (property "Datasheet" "" (id 3) (at 318.77 85.09 0)
+      (effects (font (size 1.27 1.27)) hide)
+    )
+    (property "Description" "3.5MM SCREW HOLE_WITHOUT NET" (id 4) (at 318.77 85.09 0)
+      (effects (font (size 1.27 1.27)) hide)
+    )
+  )
+  (symbol (lib_id "HandyRadio:HEADPHONE") (at 107.95 151.13 0) (unit 1)
+    (in_bom yes) (on_board yes) (fields_autoplaced)
+    (property "Reference" "LS1" (id 0) (at 135.89 156.2099 0)
+      (effects (font (size 1.27 1.27)) (justify left))
+    )
+    (property "Value" "HEADPHONE" (id 1) (at 135.89 158.7499 0)
+      (effects (font (size 1.27 1.27)) (justify left))
+    )
+    (property "Footprint" "" (id 2) (at 114.3 142.24 0)
+      (effects (font (size 1.27 1.27)) hide)
+    )
+    (property "Datasheet" "https://www.amazon.ca/JBL-Endurance-Headphone-one-Button-Remote/dp/B07NVXJNHG/ref=sr_1_10?keywords=headphone%2Bwired&qid=1665511384&qu=eyJxc2MiOiI1LjMyIiwicXNhIjoiNS4xNiIsInFzcCI6IjQuNTcifQ%3D%3D&sprefix=headphone%2Bwir%2Caps%2C399&sr=8-10&th=1" (id 3) (at 114.3 142.24 0)
+      (effects (font (size 1.27 1.27)) hide)
+    )
+    (property "Description" "JBL Endurance Run Wired Sweatproof In-Ear Sport Headphones" (id 4) (at 114.3 142.24 0)
+      (effects (font (size 1.27 1.27)) hide)
+    )
+  )
+  (symbol (lib_id "HandyRadio:SCREW_HOLE") (at 287.02 90.17 0) (unit 1)
+    (in_bom no) (on_board yes) (fields_autoplaced)
+    (property "Reference" "H3" (id 0) (at 292.1 88.8999 0)
+      (effects (font (size 1.27 1.27)) (justify left))
+    )
+    (property "Value" "SCREW_HOLE" (id 1) (at 292.1 91.4399 0)
+      (effects (font (size 1.27 1.27)) (justify left))
+    )
+    (property "Footprint" "" (id 2) (at 294.64 85.09 0)
+      (effects (font (size 1.27 1.27)) hide)
+    )
+    (property "Datasheet" "" (id 3) (at 294.64 85.09 0)
+      (effects (font (size 1.27 1.27)) hide)
+    )
+    (property "Description" "3.5MM SCREW HOLE_WITHOUT NET" (id 4) (at 294.64 85.09 0)
+      (effects (font (size 1.27 1.27)) hide)
+    )
+  )
+  (symbol (lib_id "HandyRadio:BOX") (at 111.76 217.17 0) (unit 1)
+    (in_bom yes) (on_board no) (fields_autoplaced)
+    (property "Reference" "H1" (id 0) (at 135.89 220.52 0)
+      (effects (font (size 1.27 1.27)) (justify left))
+    )
+    (property "Value" "BOX" (id 1) (at 135.89 223.06 0)
+      (effects (font (size 1.27 1.27)) (justify left))
+    )
+    (property "Footprint" "" (id 2) (at 111.76 217.17 0)
+      (effects (font (size 1.27 1.27)) hide)
+    )
+    (property "Datasheet" "" (id 3) (at 111.76 217.17 0)
+      (effects (font (size 1.27 1.27)) hide)
+    )
+    (property "Description" "3D-BOX THAT WILL DESIGN WITH FREECAD" (id 4) (at 111.76 217.17 0)
+      (effects (font (size 1.27 1.27)) hide)
+    )
+  )
+  (symbol (lib_id "HandyRadio:FERRITE_ANTENNA") (at 111.76 177.8 0) (unit 1)
+    (in_bom yes) (on_board yes) (fields_autoplaced)
+    (property "Reference" "ANT2" (id 0) (at 122.555 172.72 0))
+    (property "Value" "FERRITE_ANTENNA" (id 1) (at 122.555 175.26 0))
+    (property "Footprint" "" (id 2) (at 120.65 171.45 0)
+      (effects (font (size 1.27 1.27)) hide)
+    )
+    (property "Datasheet" "" (id 3) (at 120.65 171.45 0)
+      (effects (font (size 1.27 1.27)) hide)
+    )
+    (property "Description" "DIA = 3MM, LENGTH = 25MM, TURNS = 110, ABOUT 450 uH" (id 4) (at 114.3 173.99 0)
+      (effects (font (size 1.27 1.27)) hide)
+    )
+  )
+  (symbol (lib_id "HandyRadio:PCB") (at 107.95 76.2 0) (unit 1)
+    (in_bom yes) (on_board no) (fields_autoplaced)
+    (property "Reference" "PCB1" (id 0) (at 134.62 87.6299 0)
+      (effects (font (size 1.27 1.27)) (justify left))
+    )
+    (property "Value" "PCB" (id 1) (at 134.62 90.1699 0)
+      (effects (font (size 1.27 1.27)) (justify left))
+    )
+    (property "Footprint" "" (id 2) (at 109.22 73.66 0)
+      (effects (font (size 1.27 1.27)) hide)
+    )
+    (property "Datasheet" "" (id 3) (at 109.22 73.66 0)
+      (effects (font (size 1.27 1.27)) hide)
+    )
+  )
+  (symbol (lib_id "HandyRadio:OLED") (at 107.95 116.84 0) (unit 1)
+    (in_bom yes) (on_board no) (fields_autoplaced)
+    (property "Reference" "DIS1" (id 0) (at 134.62 128.2699 0)
+      (effects (font (size 1.27 1.27)) (justify left))
+    )
+    (property "Value" "OLED" (id 1) (at 134.62 130.8099 0)
+      (effects (font (size 1.27 1.27)) (justify left))
+    )
+    (property "Footprint" "" (id 2) (at 111.76 111.76 0)
+      (effects (font (size 1.27 1.27)) hide)
+    )
+    (property "Datasheet" "https://media.digikey.com/pdf/Data%20Sheets/Adafruit%20PDFs/938_Web.pdf" (id 3) (at 111.76 111.76 0)
+      (effects (font (size 1.27 1.27)) hide)
+    )
+    (property "Description" "Graphic LCD Display Module Passive White OLED - Passive Matrix I²C, SPI 1.3\" (33.02mm) 128 x 64" (id 4) (at 111.76 111.76 0)
+      (effects (font (size 1.27 1.27)) hide)
+    )
   )
 )

Commit message: almost ready for routing and finishing PCB :D
Parts:
- removed H2, H3, H4, H5: SCREW_HOLE, symbol HandyRadio:SCREW_HOLE
- added H2, H3, H4, H5: MOUNTING_HOLE, MountingHole:MountingHole_3.2mm_M3, symbol HandyRadio:MOUNTING_HOLE
- renumbered ANT2 to ANT1
Changed lines of the file:
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@@
     )
   )
-  (symbol (lib_id "HandyRadio:SCREW_HOLE") (at 287.02 78.74 0) (unit 1)
+  (symbol (lib_id "HandyRadio:MOUNTING_HOLE") (at 312.42 92.71 0) (unit 1)
     (in_bom no) (on_board yes) (fields_autoplaced)
-    (property "Reference" "H2" (id 0) (at 292.1 77.4699 0)
+    (property "Reference" "H5" (id 0) (at 317.5 91.4399 0)
       (effects (font (size 1.27 1.27)) (justify left))
     )
-    (property "Value" "SCREW_HOLE" (id 1) (at 292.1 80.0099 0)
+    (property "Value" "MOUNTING_HOLE" (id 1) (at 317.5 93.9799 0)
       (effects (font (size 1.27 1.27)) (justify left))
     )
-    (property "Footprint" "" (id 2) (at 294.64 73.66 0)
+    (property "Footprint" "MountingHole:MountingHole_3.2mm_M3" (id 2) (at 318.77 81.28 0)
       (effects (font (size 1.27 1.27)) hide)
     )
-    (property "Datasheet" "" (id 3) (at 294.64 73.66 0)
+    (property "Datasheet" "" (id 3) (at 320.04 87.63 0)
       (effects (font (size 1.27 1.27)) hide)
     )
-    (property "Description" "3.5MM SCREW HOLE_WITHOUT NET" (id 4) (at 294.64 73.66 0)
+    (property "Description" "M3 MOUNTING HOLE_WITHOUT NET" (id 4) (at 318.77 83.82 0)
       (effects (font (size 1.27 1.27)) hide)
     )
   )
-  (symbol (lib_id "HandyRadio:SCREW_HOLE") (at 311.15 78.74 0) (unit 1)
+  (symbol (lib_id "HandyRadio:MOUNTING_HOLE") (at 312.42 80.01 0) (unit 1)
     (in_bom no) (on_board yes) (fields_autoplaced)
-    (property "Reference" "H4" (id 0) (at 316.23 77.4699 0)
+    (property "Reference" "H4" (id 0) (at 317.5 78.7399 0)
       (effects (font (size 1.27 1.27)) (justify left))
     )
-    (property "Value" "SCREW_HOLE" (id 1) (at 316.23 80.0099 0)
+    (property "Value" "MOUNTING_HOLE" (id 1) (at 317.5 81.2799 0)
       (effects (font (size 1.27 1.27)) (justify left))
     )
-    (property "Footprint" "" (id 2) (at 318.77 73.66 0)
+    (property "Footprint" "MountingHole:MountingHole_3.2mm_M3" (id 2) (at 318.77 68.58 0)
       (effects (font (size 1.27 1.27)) hide)
     )
-    (property "Datasheet" "" (id 3) (at 318.77 73.66 0)
+    (property "Datasheet" "" (id 3) (at 320.04 74.93 0)
       (effects (font (size 1.27 1.27)) hide)
     )
-    (property "Description" "3.5MM SCREW HOLE_WITHOUT NET" (id 4) (at 318.77 73.66 0)
-      (effects (font (size 1.27 1.27)) hide)
-    )
-  )
-  (symbol (lib_id "HandyRadio:SCREW_HOLE") (at 311.15 90.17 0) (unit 1)
-    (in_bom no) (on_board yes) (fields_autoplaced)
-    (property "Reference" "H5" (id 0) (at 316.23 88.8999 0)
-      (effects (font (size 1.27 1.27)) (justify left))
-    )
-    (property "Value" "SCREW_HOLE" (id 1) (at 316.23 91.4399 0)
-      (effects (font (size 1.27 1.27)) (justify left))
-    )
-    (property "Footprint" "" (id 2) (at 318.77 85.09 0)
-      (effects (font (size 1.27 1.27)) hide)
-    )
-    (property "Datasheet" "" (id 3) (at 318.77 85.09 0)
-      (effects (font (size 1.27 1.27)) hide)
-    )
-    (property "Description" "3.5MM SCREW HOLE_WITHOUT NET" (id 4) (at 318.77 85.09 0)
+    (property "Description" "M3 MOUNTING HOLE_WITHOUT NET" (id 4) (at 318.77 71.12 0)
       (effects (font (size 1.27 1.27)) hide)
     )
@@
     )
   )
-  (symbol (lib_id "HandyRadio:SCREW_HOLE") (at 287.02 90.17 0) (unit 1)
+  (symbol (lib_id "HandyRadio:MOUNTING_HOLE") (at 283.21 80.01 0) (unit 1)
     (in_bom no) (on_board yes) (fields_autoplaced)
-    (property "Reference" "H3" (id 0) (at 292.1 88.8999 0)
+    (property "Reference" "H2" (id 0) (at 288.29 78.7399 0)
       (effects (font (size 1.27 1.27)) (justify left))
     )
-    (property "Value" "SCREW_HOLE" (id 1) (at 292.1 91.4399 0)
+    (property "Value" "MOUNTING_HOLE" (id 1) (at 288.29 81.2799 0)
       (effects (font (size 1.27 1.27)) (justify left))
     )
-    (property "Footprint" "" (id 2) (at 294.64 85.09 0)
+    (property "Footprint" "MountingHole:MountingHole_3.2mm_M3" (id 2) (at 289.56 68.58 0)
       (effects (font (size 1.27 1.27)) hide)
     )
-    (property "Datasheet" "" (id 3) (at 294.64 85.09 0)
+    (property "Datasheet" "" (id 3) (at 290.83 74.93 0)
       (effects (font (size 1.27 1.27)) hide)
     )
-    (property "Description" "3.5MM SCREW HOLE_WITHOUT NET" (id 4) (at 294.64 85.09 0)
+    (property "Description" "M3 MOUNTING HOLE_WITHOUT NET" (id 4) (at 289.56 71.12 0)
       (effects (font (size 1.27 1.27)) hide)
     )
@@
     )
   )
+  (symbol (lib_id "HandyRadio:MOUNTING_HOLE") (at 283.21 92.71 0) (unit 1)
+    (in_bom no) (on_board yes) (fields_autoplaced)
+    (property "Reference" "H3" (id 0) (at 288.29 91.4399 0)
+      (effects (font (size 1.27 1.27)) (justify left))
+    )
+    (property "Value" "MOUNTING_HOLE" (id 1) (at 288.29 93.9799 0)
+      (effects (font (size 1.27 1.27)) (justify left))
+    )
+    (property "Footprint" "MountingHole:MountingHole_3.2mm_M3" (id 2) (at 289.56 81.28 0)
+      (effects (font (size 1.27 1.27)) hide)
+    )
+    (property "Datasheet" "" (id 3) (at 290.83 87.63 0)
+      (effects (font (size 1.27 1.27)) hide)
+    )
+    (property "Description" "M3 MOUNTING HOLE_WITHOUT NET" (id 4) (at 289.56 83.82 0)
+      (effects (font (size 1.27 1.27)) hide)
+    )
+  )
   (symbol (lib_id "HandyRadio:FERRITE_ANTENNA") (at 111.76 177.8 0) (unit 1)
     (in_bom yes) (on_board yes) (fields_autoplaced)
-    (property "Reference" "ANT2" (id 0) (at 122.555 172.72 0))
+    (property "Reference" "ANT1" (id 0) (at 122.555 172.72 0))
     (property "Value" "FERRITE_ANTENNA" (id 1) (at 122.555 175.26 0))
     (property "Footprint" "" (id 2) (at 120.65 171.45 0)

Commit message: Working on lib and pcb layout
Parts:
- DIS1: footprint (none) -> _HW_HandyRadio_Footprint:OLED 1.3INCH
Changed lines of the file:
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@@
+    )
+  )
+  (symbol (lib_id "HandyRadio:OLED") (at 107.95 114.3 0) (unit 1)
+    (in_bom yes) (on_board yes) (fields_autoplaced)
+    (property "Reference" "DIS1" (id 0) (at 134.62 125.7299 0)
+      (effects (font (size 1.27 1.27)) (justify left))
+    )
+    (property "Value" "OLED" (id 1) (at 134.62 128.2699 0)
+      (effects (font (size 1.27 1.27)) (justify left))
+    )
+    (property "Footprint" "_HW_HandyRadio_Footprint:OLED 1.3INCH" (id 2) (at 111.76 109.22 0)
+      (effects (font (size 1.27 1.27)) hide)
+    )
+    (property "Datasheet" "https://media.digikey.com/pdf/Data%20Sheets/Adafruit%20PDFs/938_Web.pdf" (id 3) (at 111.76 105.41 0)
+      (effects (font (size 1.27 1.27)) hide)
+    )
+    (property "Description" "Graphic LCD Display Module Passive White OLED - Passive Matrix I²C, SPI 1.3\" (33.02mm) 128 x 64" (id 4) (at 113.03 102.87 0)
+      (effects (font (size 1.27 1.27)) hide)
     )
   )
@@
       (effects (font (size 1.27 1.27)) hide)
     )
-  )
-  (symbol (lib_id "HandyRadio:OLED") (at 107.95 116.84 0) (unit 1)
-    (in_bom yes) (on_board no) (fields_autoplaced)
-    (property "Reference" "DIS1" (id 0) (at 134.62 128.2699 0)
-      (effects (font (size 1.27 1.27)) (justify left))
-    )
-    (property "Value" "OLED" (id 1) (at 134.62 130.8099 0)
-      (effects (font (size 1.27 1.27)) (justify left))
-    )
-    (property "Footprint" "" (id 2) (at 111.76 111.76 0)
-      (effects (font (size 1.27 1.27)) hide)
-    )
-    (property "Datasheet" "https://media.digikey.com/pdf/Data%20Sheets/Adafruit%20PDFs/938_Web.pdf" (id 3) (at 111.76 111.76 0)
-      (effects (font (size 1.27 1.27)) hide)
-    )
-    (property "Description" "Graphic LCD Display Module Passive White OLED - Passive Matrix I²C, SPI 1.3\" (33.02mm) 128 x 64" (id 4) (at 111.76 111.76 0)
-      (effects (font (size 1.27 1.27)) hide)
-    )

Commit message: serious modification has been done
Parts:
- removed LS1: HEADPHONE, symbol HandyRadio:HEADPHONE
- added SPK1: SPEAKER-8OHM, symbol HandyRadio:SPEAKER-8OHM
Changed lines of the file:
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@@
-    )
-  )
-  (symbol (lib_id "HandyRadio:HEADPHONE") (at 107.95 151.13 0) (unit 1)
-    (in_bom yes) (on_board yes) (fields_autoplaced)
-    (property "Reference" "LS1" (id 0) (at 135.89 156.2099 0)
-      (effects (font (size 1.27 1.27)) (justify left))
-    )
-    (property "Value" "HEADPHONE" (id 1) (at 135.89 158.7499 0)
-      (effects (font (size 1.27 1.27)) (justify left))
-    )
-    (property "Footprint" "" (id 2) (at 114.3 142.24 0)
-      (effects (font (size 1.27 1.27)) hide)
-    )
-    (property "Datasheet" "https://www.amazon.ca/JBL-Endurance-Headphone-one-Button-Remote/dp/B07NVXJNHG/ref=sr_1_10?keywords=headphone%2Bwired&qid=1665511384&qu=eyJxc2MiOiI1LjMyIiwicXNhIjoiNS4xNiIsInFzcCI6IjQuNTcifQ%3D%3D&sprefix=headphone%2Bwir%2Caps%2C399&sr=8-10&th=1" (id 3) (at 114.3 142.24 0)
-      (effects (font (size 1.27 1.27)) hide)
-    )
-    (property "Description" "JBL Endurance Run Wired Sweatproof In-Ear Sport Headphones" (id 4) (at 114.3 142.24 0)
-      (effects (font (size 1.27 1.27)) hide)
     )
   )
@@
       (effects (font (size 1.27 1.27)) hide)
     )
+  )
+  (symbol (lib_id "HandyRadio:SPEAKER-8OHM") (at 109.22 143.51 0) (unit 1)
+    (in_bom yes) (on_board no) (fields_autoplaced)
+    (property "Reference" "SPK1" (id 0) (at 134.62 154.9399 0)
+      (effects (font (size 1.27 1.27)) (justify left))
+    )
+    (property "Value" "SPEAKER-8OHM" (id 1) (at 134.62 157.4799 0)
+      (effects (font (size 1.27 1.27)) (justify left))
+    )
+    (property "Footprint" "" (id 2) (at 109.22 143.51 0)
+      (effects (font (size 1.27 1.27)) hide)
+    )
+    (property "Datasheet" "https://www.cuidevices.com/product/resource/cls0201ma.pdf" (id 3) (at 116.84 138.43 0)
+      (effects (font (size 1.27 1.27)) hide)
+    )
+    (property "Description" "SPEAKER 8OHM .5W 20MM ROUND" (id 4) (at 115.57 135.89 0)
+      (effects (font (size 1.27 1.27)) hide)
+    )

Commit message: IT'S ALMOST GOOD FOR RELEASE, schematic should be checked and a double check on routing
Parts:
- H2, H3, H4, H5: footprint MountingHole:MountingHole_3.2mm_M3 -> _HW_HandyRadio_Footprint:MountingHole_3.2mm_M3
Changed lines of the file:
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@@
       (effects (font (size 1.27 1.27)) (justify left))
     )
-    (property "Footprint" "MountingHole:MountingHole_3.2mm_M3" (id 2) (at 318.77 81.28 0)
+    (property "Footprint" "_HW_HandyRadio_Footprint:MountingHole_3.2mm_M3" (id 2) (at 318.77 81.28 0)
       (effects (font (size 1.27 1.27)) hide)
     )
@@
     )
   )
-  (symbol (lib_id "HandyRadio:MOUNTING_HOLE") (at 312.42 80.01 0) (unit 1)
+  (symbol (lib_name "MOUNTING_HOLE_2") (lib_id "HandyRadio:MOUNTING_HOLE") (at 312.42 80.01 0) (unit 1)
     (in_bom no) (on_board yes) (fields_autoplaced)
     (property "Reference" "H4" (id 0) (at 317.5 78.7399 0)
@@
       (effects (font (size 1.27 1.27)) (justify left))
     )
-    (property "Footprint" "MountingHole:MountingHole_3.2mm_M3" (id 2) (at 318.77 68.58 0)
+    (property "Footprint" "_HW_HandyRadio_Footprint:MountingHole_3.2mm_M3" (id 2) (at 318.77 68.58 0)
       (effects (font (size 1.27 1.27)) hide)
     )
@@
     )
   )
-  (symbol (lib_id "HandyRadio:MOUNTING_HOLE") (at 283.21 80.01 0) (unit 1)
+  (symbol (lib_name "MOUNTING_HOLE_1") (lib_id "HandyRadio:MOUNTING_HOLE") (at 283.21 80.01 0) (unit 1)
     (in_bom no) (on_board yes) (fields_autoplaced)
     (property "Reference" "H2" (id 0) (at 288.29 78.7399 0)
@@
       (effects (font (size 1.27 1.27)) (justify left))
     )
-    (property "Footprint" "MountingHole:MountingHole_3.2mm_M3" (id 2) (at 289.56 68.58 0)
+    (property "Footprint" "_HW_HandyRadio_Footprint:MountingHole_3.2mm_M3" (id 2) (at 289.56 68.58 0)
       (effects (font (size 1.27 1.27)) hide)
     )
@@
     )
   )
-  (symbol (lib_id "HandyRadio:MOUNTING_HOLE") (at 283.21 92.71 0) (unit 1)
+  (symbol (lib_name "MOUNTING_HOLE_3") (lib_id "HandyRadio:MOUNTING_HOLE") (at 283.21 92.71 0) (unit 1)
     (in_bom no) (on_board yes) (fields_autoplaced)
     (property "Reference" "H3" (id 0) (at 288.29 91.4399 0)
@@
       (effects (font (size 1.27 1.27)) (justify left))
     )
-    (property "Footprint" "MountingHole:MountingHole_3.2mm_M3" (id 2) (at 289.56 81.28 0)
+    (property "Footprint" "_HW_HandyRadio_Footprint:MountingHole_3.2mm_M3" (id 2) (at 289.56 81.28 0)
       (effects (font (size 1.27 1.27)) hide)
     )
