File: HandyRadio/HW/V1_09302022/1- Design Files/_HW_HandyRadio_/[07] - MECHANICAL PARTS.kicad_sch (KiCad schematic)
At the start: 11 parts

Commit message: some modification
Parts:
- renumbered ANT1 to ANT601, BATT1 to BATT601, DIS1 to DIS601, H1 to H601, H2 to H602, H3 to H603, H4 to H604, H5 to H605, LBL1 to LBL601, PCB1 to PCB601, SPK1 to SPK601
Changed lines of the file:
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@@
   (symbol (lib_id "HandyRadio:LABLES") (at 195.58 76.2 0) (unit 1)
     (in_bom no) (on_board no) (fields_autoplaced)
-    (property "Reference" "LBL1" (id 0) (at 238.76 82.5499 0)
+    (property "Reference" "LBL601" (id 0) (at 238.76 82.5499 0)
       (effects (font (size 1.27 1.27)) (justify left))
     )
@@
   (symbol (lib_id "HandyRadio:Li-PO_BATTERY") (at 104.14 194.31 0) (unit 1)
     (in_bom yes) (on_board yes) (fields_autoplaced)
-    (property "Reference" "BATT1" (id 0) (at 122.555 189.23 0))
+    (property "Reference" "BATT601" (id 0) (at 122.555 189.23 0))
     (property "Value" "Li-PO_BATTERY" (id 1) (at 122.555 191.77 0))
     (property "Footprint" "" (id 2) (at 109.22 185.42 0)
@@
   (symbol (lib_id "HandyRadio:MOUNTING_HOLE") (at 312.42 92.71 0) (unit 1)
     (in_bom no) (on_board yes) (fields_autoplaced)
-    (property "Reference" "H5" (id 0) (at 317.5 91.4399 0)
+    (property "Reference" "H605" (id 0) (at 317.5 91.4399 0)
       (effects (font (size 1.27 1.27)) (justify left))
     )
@@
   (symbol (lib_name "MOUNTING_HOLE_2") (lib_id "HandyRadio:MOUNTING_HOLE") (at 312.42 80.01 0) (unit 1)
     (in_bom no) (on_board yes) (fields_autoplaced)
-    (property "Reference" "H4" (id 0) (at 317.5 78.7399 0)
+    (property "Reference" "H604" (id 0) (at 317.5 78.7399 0)
       (effects (font (size 1.27 1.27)) (justify left))
     )
@@
   (symbol (lib_name "MOUNTING_HOLE_1") (lib_id "HandyRadio:MOUNTING_HOLE") (at 283.21 80.01 0) (unit 1)
     (in_bom no) (on_board yes) (fields_autoplaced)
-    (property "Reference" "H2" (id 0) (at 288.29 78.7399 0)
+    (property "Reference" "H602" (id 0) (at 288.29 78.7399 0)
       (effects (font (size 1.27 1.27)) (justify left))
     )
@@
   (symbol (lib_id "HandyRadio:BOX") (at 111.76 217.17 0) (unit 1)
     (in_bom yes) (on_board no) (fields_autoplaced)
-    (property "Reference" "H1" (id 0) (at 135.89 220.52 0)
+    (property "Reference" "H601" (id 0) (at 135.89 220.52 0)
       (effects (font (size 1.27 1.27)) (justify left))
     )
@@
   (symbol (lib_name "MOUNTING_HOLE_3") (lib_id "HandyRadio:MOUNTING_HOLE") (at 283.21 92.71 0) (unit 1)
     (in_bom no) (on_board yes) (fields_autoplaced)
-    (property "Reference" "H3" (id 0) (at 288.29 91.4399 0)
+    (property "Reference" "H603" (id 0) (at 288.29 91.4399 0)
       (effects (font (size 1.27 1.27)) (justify left))
     )
@@
   (symbol (lib_id "HandyRadio:FERRITE_ANTENNA") (at 111.76 177.8 0) (unit 1)
     (in_bom yes) (on_board yes) (fields_autoplaced)
-    (property "Reference" "ANT1" (id 0) (at 122.555 172.72 0))
+    (property "Reference" "ANT601" (id 0) (at 122.555 172.72 0))
     (property "Value" "FERRITE_ANTENNA" (id 1) (at 122.555 175.26 0))
     (property "Footprint" "" (id 2) (at 120.65 171.45 0)
@@
   (symbol (lib_id "HandyRadio:OLED") (at 107.95 114.3 0) (unit 1)
     (in_bom yes) (on_board yes) (fields_autoplaced)
-    (property "Reference" "DIS1" (id 0) (at 134.62 125.7299 0)
+    (property "Reference" "DIS601" (id 0) (at 134.62 125.7299 0)
       (effects (font (size 1.27 1.27)) (justify left))
     )
@@
   (symbol (lib_id "HandyRadio:PCB") (at 107.95 76.2 0) (unit 1)
     (in_bom yes) (on_board no) (fields_autoplaced)
-    (property "Reference" "PCB1" (id 0) (at 134.62 87.6299 0)
+    (property "Reference" "PCB601" (id 0) (at 134.62 87.6299 0)
       (effects (font (size 1.27 1.27)) (justify left))
     )
@@
   (symbol (lib_id "HandyRadio:SPEAKER-8OHM") (at 109.22 143.51 0) (unit 1)
     (in_bom yes) (on_board no) (fields_autoplaced)
-    (property "Reference" "SPK1" (id 0) (at 134.62 154.9399 0)
+    (property "Reference" "SPK601" (id 0) (at 134.62 154.9399 0)
       (effects (font (size 1.27 1.27)) (justify left))
     )

Commit message: replacement almost done, but routing left
Parts:
- added LBL602: Mend0z0_LOGO, _HW_HandyRadio_Footprint:Logo, symbol HandyRadio:Mend0z0_LOGO
Changed lines of the file:
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@@
+    )
+  )
+  (symbol (lib_id "HandyRadio:Mend0z0_LOGO") (at 198.12 105.41 0) (unit 1)
+    (in_bom no) (on_board yes) (fields_autoplaced)
+    (property "Reference" "LBL602" (id 0) (at 209.55 108.2674 0)
+      (effects (font (size 1.27 1.27)) (justify left))
+    )
+    (property "Value" "Mend0z0_LOGO" (id 1) (at 209.55 110.8074 0)
+      (effects (font (size 1.27 1.27)) (justify left))
+    )
+    (property "Footprint" "_HW_HandyRadio_Footprint:Logo" (id 2) (at 213.36 100.965 0)
+      (effects (font (size 1.27 1.27)) hide)
+    )
+    (property "Datasheet" "" (id 3) (at 198.12 105.41 0)
+      (effects (font (size 1.27 1.27)) hide)
     )
   )
