File: HandyRadio/HW/V1_09302022/1- Design Files/_HW_HandyRadio_/[07] - MECHANICAL PARTS.kicad_sch (KiCad schematic)
At the start: 12 parts

Commit message: Ready to release the HW :smile:
Other:
- note added: "CHECKED"
Changed lines of the file:
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@@
   (title_block
     (title "Handy Radio")
+    (date "2022-11-10")
     (rev "01")
     (company "Siavash Taher Parvar")
@@
     (comment 9 "N/A")
   )
+  (text "CHECKED" (at 378.46 38.1 0)
+    (effects (font (size 5 5) (thickness 1) bold) (justify left bottom))
+  )
   (symbol (lib_id "HandyRadio:LABLES") (at 195.58 76.2 0) (unit 1)
