File: HandyRadio/HW/V1_09302022/1- Design Files/_HW_HandyRadio_/[02] - BLOCK DIAGRAM.kicad_sch (KiCad schematic)
At the start: 0 parts

Commit message: HandyRadio BlockDiagram has been done
Other:
- note added: "3X PUSHBUTTONS"
- note added: "AM/LW ANTENNA"
- note added: "AUDIO AMP"
- note added: "BATT CHARGER"
- note added: "DC/DC BOOST +5.5VDC"
- note added: "FM/AM/LW/SW RECEIVER"
- note added: "GPIO"
- note added: "HEADPHONE (FM/SW ANT)"
- note added: "I2C"
- note added: "LDO +3.3VDC"
- note added: "LED"
- note added: "Li-ion Battery +3.7VDC"
- note added: "MCU RTC"
- note added: "OLED"
- note added: "PWM"
- note added: "Page 03"
- note added: "Page 04"
- note added: "Page 05"
- note added: "Page 06"
- note added: "STEREO OUT"

Commit message: 1/6 of the hardware has been done
Other:
- note added: "IR INPUT"

Commit message: Schematic is almost Done
Other:
- company: (none) -> Siavash Taher Parvar
- title: (none) -> Handy Radio
Changed lines of the file:
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@@
 (kicad_sch (version 20211123) (generator eeschema)
   (paper "B")
+  (title_block
+    (title "Handy Radio")
+    (rev "01")
+    (company "Siavash Taher Parvar")
+    (comment 1 "Siavash Taher Parvar")
+    (comment 2 "Siavash Taher Parvar")
+    (comment 3 "Siavash Taher Parvar")
+    (comment 4 "N/A")
+    (comment 5 "N/A")
+    (comment 6 "N/A")
+    (comment 8 "NO VARIANT")
+    (comment 9 "N/A")
+  )
   (polyline (pts (xy 190.5 241.3) (xy 165.1 241.3))
     (stroke (width 0) (type default) (color 0 0 0 0))

Commit message: Schematic has been double checked
Other:
- note added: "ADC"
Changed lines of the file:
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@@
+    (stroke (width 0) (type default) (color 0 0 0 0))
+  )
+  (polyline (pts (xy 63.5 215.9) (xy 63.5 208.28))
+    (stroke (width 0) (type default) (color 0 0 0 0))
+  )
+  (polyline (pts (xy 184.15 208.28) (xy 184.15 144.78))
     (stroke (width 0) (type default) (color 0 0 0 0))
   )
@@
     (stroke (width 0) (type default) (color 0 0 0 0))
   )
+  (polyline (pts (xy 184.15 144.78) (xy 196.85 144.78))
+    (stroke (width 0) (type default) (color 0 0 0 0))
+  )
   (polyline (pts (xy 292.1 114.3) (xy 292.1 139.7))
     (stroke (width 0) (type default) (color 0 0 0 0))
@@
     (stroke (width 0) (type default) (color 0 0 0 0))
   )
+  (polyline (pts (xy 63.5 208.28) (xy 184.15 208.28))
+    (stroke (width 0) (type default) (color 0 0 0 0))
+  )
   (polyline (pts (xy 279.4 107.95) (xy 254 107.95))
     (stroke (width 0) (type default) (color 0 0 0 0))
@@
     (effects (font (size 1.27 1.27)) (justify left bottom))
   )
-  (text "GPIO" (at 187.96 139.7 0)
+  (text "GPIO" (at 189.23 139.7 0)
     (effects (font (size 2 2)) (justify left bottom))
   )
@@
     (effects (font (size 2 2)) (justify left bottom))
   )
+  (text "ADC" (at 190.5 144.78 0)
+    (effects (font (size 2 2)) (justify left bottom))
+  )

Commit message: almost ready for routing and finishing PCB :D
Other:
- added sheet AUDIO AMP ([05] - AUDIO AMP.kicad_sch)
- added sheet DCDC PWS ([06] - DCDC PWS.kicad_sch)
- added sheet MCU, RTC, OLED, PB, LED ([03] - MCU, RTC, OLED, PB, LED.kicad_sch)
- added sheet RF RECEIVER ([04] - RF RECEIVER.kicad_sch)
- note removed: "HEADPHONE (FM/SW ANT)"

Commit message: serious modification has been done
Other:
- note added: "LDO +5VDC"
- note added: "MONO AUDIO AMP"
- note removed: "AM/LW ANTENNA"
- note removed: "AUDIO AMP"
- note removed: "FM/AM/LW/SW RECEIVER"

Commit message: Ready to release the HW :smile:
Other:
- note added: "CHECKED"
Changed lines of the file:
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@@
   (title_block
     (title "Handy Radio")
+    (date "2022-11-10")
     (rev "01")
     (company "Siavash Taher Parvar")
@@
     (effects (font (size 1.27 1.27)) (justify left bottom))
   )
+  (text "CHECKED" (at 379.73 38.1 0)
+    (effects (font (size 5 5) (thickness 1) bold) (justify left bottom))
+  )
   (text "LED" (at 276.86 166.37 0)
