File: HandyRadio/HW/V1_09302022/1- Design Files/_HW_HandyRadio_/[08] - REVISION HISTORY.kicad_sch (KiCad schematic)
At the start: 0 parts

Commit message: Schematic is almost Done
Other:
- note removed: "add an OLED display add a Ferrite bead antenna add a earpod add a lithium battery add a box add a PCB add labels"
Changed lines of the file:
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@@
     (comment 9 "N/A")
   )
-  (text "add an OLED display\n\nadd a Ferrite bead antenna\n\nadd a earpod\n\nadd a lithium battery\n\nadd a box\n\nadd a PCB\n\nadd labels"
-    (at 134.62 163.83 0)
-    (effects (font (size 3 3)) (justify left bottom))
-  )
 )

Commit message: Ready to release the HW :smile:
Other:
- note added: "CHECKED"
Changed lines of the file:
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@@
   (title_block
     (title "Handy Radio")
+    (date "2022-11-10")
     (rev "01")
     (company "Siavash Taher Parvar")
@@
     (comment 9 "N/A")
   )
+  (text "CHECKED" (at 379.73 38.1 0)
+    (effects (font (size 5 5) (thickness 1) bold) (justify left bottom))
+  )
 )
